File: Goku _ Vegeta/3.0/Line 3.0 - GV3/Line 3.0.kicad_pcb (KiCad board)
At the start: 2 copper layers, 215 x 206.6 mm, 58 parts, among them J1 I2C MAIN, J2 LEFT HEADERS, J3 RIGHT HEADERS, U1 DEV-16771, U2 NXV55UNR

Commit message: sumonyx code
need to get
Parts:
- removed A1, A10, A11, A12, A2, A3, A4, A5, A6, A7, A8, A9: ALS-PT19-315C/L177/TR8, ALS-PT19-315C_L177_TR8:XDCR_ALS-PT19-315C_L177_TR8
- removed G*** (x4): LOGO, LOGO
- removed J1: I2C MAIN, Connector_JST:JST_XH_B3B-XH-A_1x03_P2.50mm_Vertical
- removed J2: LEFT HEADERS, Connector_PinHeader_2.54mm:PinHeader_1x24_P2.54mm_Vertical
- removed J3: RIGHT HEADERS, Connector_PinHeader_2.54mm:PinHeader_1x24_P2.54mm_Vertical
- removed LED1, LED10, LED11, LED12, LED2, LED3, LED4, LED5, LED6, LED7, LED8, LED9: JB2835AWT-W-U30GA0000-N0000001, JB2835AWT-W-U30GA0000-N0000001:LED_J2835_CRW
- removed R1, R11, R13, R15, R17, R19, R21, R23, R3, R5, R7, R9: 36R, Resistor_SMD:R_0805_2012Metric
- removed R10, R12, R14, R16, R18, R2, R20, R22, R24, R25, R4, R6, R8: 10K, Resistor_SMD:R_0805_2012Metric
- removed U1: DEV-16771, DEV-16771:MODULE_DEV-16771
- removed U2: NXV55UNR, NXV55UNR:TRANS_BC846B,215
Routing:
- net +5V: track 1695.0 -> 0.00 mm, vias 12 -> 0
- net (no net): track 566.6 -> 0.00 mm, vias 8 -> 0
- net GND: track 26.2 -> 0.00 mm, vias 12 -> 0
Other:
- board outline removed
- board text removed: "Designed by Hugh Phan 9/07/2023"
- board text removed: "Fort Street Team Silverback 2023 Hugh Phan Issey Lee Jayden Nguyen Jack Sumner K.Z"
- board text removed: "G V 2"
- board text removed: "LINE 2.4 PCB"

Commit message: Started 3.1 PCBs
Parts:
- added A1: ALS-PT19-315C/L177/TR8, ALS-PT19-315C_L177_TR8:XDCR_ALS-PT19-315C_L177_TR8, F.Cu at (81.1, 139.8)
- added A10: ALS-PT19-315C/L177/TR8, ALS-PT19-315C_L177_TR8:XDCR_ALS-PT19-315C_L177_TR8, F.Cu at (85.5, 146.8)
- added A11: ALS-PT19-315C/L177/TR8, ALS-PT19-315C_L177_TR8:XDCR_ALS-PT19-315C_L177_TR8, F.Cu at (85.5, 149.2)
- added A12: ALS-PT19-315C/L177/TR8, ALS-PT19-315C_L177_TR8:XDCR_ALS-PT19-315C_L177_TR8, F.Cu at (85.5, 151.6)
- added A13: ALS-PT19-315C/L177/TR8, ALS-PT19-315C_L177_TR8:XDCR_ALS-PT19-315C_L177_TR8, F.Cu at (89.8, 139.8)
- added A14: ALS-PT19-315C/L177/TR8, ALS-PT19-315C_L177_TR8:XDCR_ALS-PT19-315C_L177_TR8, F.Cu at (89.8, 142.2)
- added A15: ALS-PT19-315C/L177/TR8, ALS-PT19-315C_L177_TR8:XDCR_ALS-PT19-315C_L177_TR8, F.Cu at (89.8, 144.5)
- added A16: ALS-PT19-315C/L177/TR8, ALS-PT19-315C_L177_TR8:XDCR_ALS-PT19-315C_L177_TR8, F.Cu at (89.8, 146.8)
- added A2: ALS-PT19-315C/L177/TR8, ALS-PT19-315C_L177_TR8:XDCR_ALS-PT19-315C_L177_TR8, F.Cu at (81.1, 142.2)
- added A3: ALS-PT19-315C/L177/TR8, ALS-PT19-315C_L177_TR8:XDCR_ALS-PT19-315C_L177_TR8, F.Cu at (81.1, 144.5)
- added A4: ALS-PT19-315C/L177/TR8, ALS-PT19-315C_L177_TR8:XDCR_ALS-PT19-315C_L177_TR8, F.Cu at (81.1, 146.8)
- added A5: ALS-PT19-315C/L177/TR8, ALS-PT19-315C_L177_TR8:XDCR_ALS-PT19-315C_L177_TR8, F.Cu at (81.1, 149.2)
- added A6: ALS-PT19-315C/L177/TR8, ALS-PT19-315C_L177_TR8:XDCR_ALS-PT19-315C_L177_TR8, F.Cu at (81.1, 151.6)
- added A7: ALS-PT19-315C/L177/TR8, ALS-PT19-315C_L177_TR8:XDCR_ALS-PT19-315C_L177_TR8, F.Cu at (85.5, 139.8)
- added A8: ALS-PT19-315C/L177/TR8, ALS-PT19-315C_L177_TR8:XDCR_ALS-PT19-315C_L177_TR8, F.Cu at (85.5, 142.2)
- added A9: ALS-PT19-315C/L177/TR8, ALS-PT19-315C_L177_TR8:XDCR_ALS-PT19-315C_L177_TR8, F.Cu at (85.5, 144.5)
- added C1: 100uF, Capacitor_THT:CP_Radial_D10.0mm_P5.00mm, F.Cu at (142.0, 105.3)
- added C10: 0.1uF, Capacitor_SMD:C_0805_2012Metric, F.Cu at (105.4, 148.3)
- added C15: 10uF, Capacitor_SMD:C_0805_2012Metric, F.Cu at (105.4, 151.3)
- added C16: 0.1uF, Capacitor_SMD:C_0805_2012Metric, F.Cu at (105.4, 154.3)
- added C17: 3.3nF, Capacitor_SMD:C_0805_2012Metric, F.Cu at (105.4, 157.4)
- added C18: 22uF, Capacitor_SMD:C_0805_2012Metric, F.Cu at (105.4, 160.4)
- added C2: 1uF, Capacitor_SMD:C_0805_2012Metric, F.Cu at (101.0, 148.3)
- added C3: 560uF, Capacitor_THT:CP_Radial_D18.0mm_P7.50mm, F.Cu at (85.2, 109.3)
- added C4: 560uF, Capacitor_THT:CP_Radial_D18.0mm_P7.50mm, F.Cu at (85.2, 128.8)
- added C5: 1uF, Capacitor_SMD:C_0805_2012Metric, F.Cu at (101.0, 151.3)
- added C6: 100uF, Capacitor_THT:CP_Radial_D10.0mm_P5.00mm, F.Cu at (142.0, 116.8)
- added C7: 22uF, Capacitor_SMD:C_0805_2012Metric, F.Cu at (101.0, 154.3)
- added C8: 10uF, Capacitor_SMD:C_0805_2012Metric, F.Cu at (101.0, 157.4)
- added C9: 3.3nF, Capacitor_SMD:C_0805_2012Metric, F.Cu at (101.0, 160.4)
- added D1: SS510, Diode_SMD:D_SOD-128, F.Cu at (134.6, 155.2)
- added D2: STTH2002G-TR, Package_TO_SOT_SMD:TO-263-2, F.Cu at (109.5, 105.7)
- added D3: STTH2002G-TR, Package_TO_SOT_SMD:TO-263-2, F.Cu at (109.5, 118.0)
- added D5: STTH2002G-TR, Package_TO_SOT_SMD:TO-263-2, F.Cu at (109.5, 130.4)
- added J1: Solenoid, TerminalBlock:TerminalBlock_bornier-2_P5.08mm, F.Cu at (141.9, 144.9)
- added J10: RIGHT HEADERS, Connector_PinHeader_2.54mm:PinHeader_1x24_P2.54mm_Vertical, F.Cu at (62.3, 101.8)
- added J11: Kicker Voltmeter, TerminalBlock:TerminalBlock_bornier-2_P5.08mm, F.Cu at (141.9, 154.0)
- added J3: Motor 1, Connector_PinSocket_2.54mm:PinSocket_1x06_P2.54mm_Vertical, F.Cu at (141.0, 125.5)
- added J4: Motor 3, Connector_PinSocket_2.54mm:PinSocket_1x06_P2.54mm_Vertical, F.Cu at (145.6, 125.5)
- added J5: Motor 2, Connector_PinSocket_2.54mm:PinSocket_1x06_P2.54mm_Vertical, F.Cu at (150.2, 125.5)
- added J6: Motor 4, Connector_PinSocket_2.54mm:PinSocket_1x06_P2.54mm_Vertical, F.Cu at (154.8, 125.5)
- added J7: BATTERY POWER, Connector_AMASS:AMASS_XT60-F_1x02_P7.20mm_Vertical, F.Cu at (103.9, 141.7)
- added J8: I2C TO MASTER, Connector_JST:JST_XH_B4B-XH-AM_1x04_P2.50mm_Vertical, F.Cu at (119.9, 156.6)
- added J9: LEFT HEADERS, Connector_PinHeader_2.54mm:PinHeader_1x24_P2.54mm_Vertical, F.Cu at (57.6, 101.8)
- added L1: 56uH, Inductor_SMD:L_Bourns_SRR1260, F.Cu at (71.6, 106.5)
- added L2: 2.2uH, Inductor_SMD:L_Bourns_SRR1260, F.Cu at (71.6, 120.6)
- added L3: 2.2uH, Inductor_SMD:L_Bourns_SRR1260, F.Cu at (71.6, 134.7)
- added LED1: JB2835AWT-W-U30GA0000-N0000001, JB2835AWT-W-U30GA0000-N0000001:LED_J2835_CRW, F.Cu at (119.2, 125.4)
- added LED10: JB2835AWT-W-U30GA0000-N0000001, JB2835AWT-W-U30GA0000-N0000001:LED_J2835_CRW, F.Cu at (130.3, 129.8)
- added LED11: JB2835AWT-W-U30GA0000-N0000001, JB2835AWT-W-U30GA0000-N0000001:LED_J2835_CRW, F.Cu at (130.3, 134.3)
- added LED12: JB2835AWT-W-U30GA0000-N0000001, JB2835AWT-W-U30GA0000-N0000001:LED_J2835_CRW, F.Cu at (130.3, 138.7)
- added LED13: JB2835AWT-W-U30GA0000-N0000001, JB2835AWT-W-U30GA0000-N0000001:LED_J2835_CRW, F.Cu at (135.9, 125.4)
- added LED14: JB2835AWT-W-U30GA0000-N0000001, JB2835AWT-W-U30GA0000-N0000001:LED_J2835_CRW, F.Cu at (135.9, 129.8)
- added LED15: JB2835AWT-W-U30GA0000-N0000001, JB2835AWT-W-U30GA0000-N0000001:LED_J2835_CRW, F.Cu at (135.9, 134.3)
- added LED16: JB2835AWT-W-U30GA0000-N0000001, JB2835AWT-W-U30GA0000-N0000001:LED_J2835_CRW, F.Cu at (135.9, 138.7)
- added LED2: JB2835AWT-W-U30GA0000-N0000001, JB2835AWT-W-U30GA0000-N0000001:LED_J2835_CRW, F.Cu at (119.2, 129.8)
- added LED3: JB2835AWT-W-U30GA0000-N0000001, JB2835AWT-W-U30GA0000-N0000001:LED_J2835_CRW, F.Cu at (119.2, 134.3)
- added LED4: JB2835AWT-W-U30GA0000-N0000001, JB2835AWT-W-U30GA0000-N0000001:LED_J2835_CRW, F.Cu at (119.2, 138.7)
- added LED5: JB2835AWT-W-U30GA0000-N0000001, JB2835AWT-W-U30GA0000-N0000001:LED_J2835_CRW, F.Cu at (124.8, 125.4)
- added LED6: JB2835AWT-W-U30GA0000-N0000001, JB2835AWT-W-U30GA0000-N0000001:LED_J2835_CRW, F.Cu at (124.8, 129.8)
- added LED7: JB2835AWT-W-U30GA0000-N0000001, JB2835AWT-W-U30GA0000-N0000001:LED_J2835_CRW, F.Cu at (124.8, 134.3)
- added LED8: JB2835AWT-W-U30GA0000-N0000001, JB2835AWT-W-U30GA0000-N0000001:LED_J2835_CRW, F.Cu at (124.8, 138.7)
- added LED9: JB2835AWT-W-U30GA0000-N0000001, JB2835AWT-W-U30GA0000-N0000001:LED_J2835_CRW, F.Cu at (130.3, 125.4)
- added Q2: BSC040N10NS5, Package_TO_SOT_SMD:TDSON-8-1, F.Cu at (93.6, 156.1)
- added R1: 2K94, Resistor_SMD:R_0805_2012Metric, F.Cu at (118.6, 101.0)
- added R10: 10K, Resistor_SMD:R_0805_2012Metric, F.Cu at (123.0, 104.0)
- added R11: 12R, Resistor_SMD:R_0805_2012Metric, F.Cu at (123.0, 106.9)
- added R12: 10K, Resistor_SMD:R_0805_2012Metric, F.Cu at (123.0, 109.8)
- added R13: 12R, Resistor_SMD:R_0805_2012Metric, F.Cu at (123.0, 112.8)
- added R14: 10K, Resistor_SMD:R_0805_2012Metric, F.Cu at (123.0, 115.8)
- added R15: 12R, Resistor_SMD:R_0805_2012Metric, F.Cu at (123.0, 118.7)
- added R16: 10K, Resistor_SMD:R_0805_2012Metric, F.Cu at (123.0, 121.7)
- added R17: 12R, Resistor_SMD:R_0805_2012Metric, F.Cu at (127.5, 101.0)
- added R18: 10K, Resistor_SMD:R_0805_2012Metric, F.Cu at (127.5, 104.0)
- added R19: 12R, Resistor_SMD:R_0805_2012Metric, F.Cu at (127.5, 106.9)
- added R2: 57K, Resistor_SMD:R_0805_2012Metric, F.Cu at (118.6, 104.0)
- added R20: 10K, Resistor_SMD:R_0805_2012Metric, F.Cu at (127.5, 109.8)
- added R21: 12R, Resistor_SMD:R_0805_2012Metric, F.Cu at (127.5, 112.8)
- added R22: 10K, Resistor_SMD:R_0805_2012Metric, F.Cu at (127.5, 115.8)
- added R23: 12R, Resistor_SMD:R_0805_2012Metric, F.Cu at (127.5, 118.7)
- added R24: 10K, Resistor_SMD:R_0805_2012Metric, F.Cu at (127.5, 121.7)
- added R25: 12R, Resistor_SMD:R_0805_2012Metric, F.Cu at (131.9, 101.0)
- added R26: 10K, Resistor_SMD:R_0805_2012Metric, F.Cu at (131.9, 104.0)
- added R27: 12R, Resistor_SMD:R_0805_2012Metric, F.Cu at (131.9, 106.9)
- added R28: 10K, Resistor_SMD:R_0805_2012Metric, F.Cu at (131.9, 109.8)
- added R29: CT6EP103, POT_CT-6EP_NDC:POT_CT-6EP_NDC, F.Cu at (82.7, 157.1)
- added R3: 1K5, Resistor_SMD:R_0805_2012Metric, F.Cu at (118.6, 106.9)
- added R30: 100K, Resistor_SMD:R_0805_2012Metric, F.Cu at (131.9, 112.8)
- added R31: 12R, Resistor_SMD:R_0805_2012Metric, F.Cu at (131.9, 115.8)
- added R32: 100K, Resistor_SMD:R_0805_2012Metric, F.Cu at (131.9, 118.7)
- added R33: 10K, Resistor_SMD:R_0805_2012Metric, F.Cu at (131.9, 121.7)
- added R34: 12R, Resistor_SMD:R_0805_2012Metric, F.Cu at (136.3, 101.0)
- added R35: 10K, Resistor_SMD:R_0805_2012Metric, F.Cu at (136.3, 104.0)
- added R36: 12R, Resistor_SMD:R_0805_2012Metric, F.Cu at (136.3, 106.9)
- added R37: 10K, Resistor_SMD:R_0805_2012Metric, F.Cu at (136.3, 109.8)
- added R38: 12R, Resistor_SMD:R_0805_2012Metric, F.Cu at (136.3, 112.8)
- added R39: 10K, Resistor_SMD:R_0805_2012Metric, F.Cu at (136.3, 115.8)
- added R4: 12R, Resistor_SMD:R_0805_2012Metric, F.Cu at (118.6, 109.8)
- added R5: 10K, Resistor_SMD:R_0805_2012Metric, F.Cu at (118.6, 112.8)
- added R6: 12R, Resistor_SMD:R_0805_2012Metric, F.Cu at (118.6, 115.8)
- added R7: 10K, Resistor_SMD:R_0805_2012Metric, F.Cu at (118.6, 118.7)
- added R8: 10K, Resistor_SMD:R_0805_2012Metric, F.Cu at (118.6, 121.7)
- added R9: 12R, Resistor_SMD:R_0805_2012Metric, F.Cu at (123.0, 101.0)
- added U1: LM2587S-ADJ, LM2587S-ADJ:VREG_TPS79625KTTR, F.Cu at (130.3, 147.1)
- added U10: TPS62132, Package_DFN_QFN:VQFN-16-1EP_3x3mm_P0.5mm_EP1.68x1.68mm_ThermalVias, F.Cu at (94.4, 141.3)
- added U11: TPS62133, Package_DFN_QFN:VQFN-16-1EP_3x3mm_P0.5mm_EP1.68x1.68mm_ThermalVias, F.Cu at (94.4, 146.6)
- added U2: TB67H420FTG Dual/Single Motor Driver Carrier, TB67H420FTG Dual_Single Motor Driver Carrier:TB67H420FTG DualSingle Motor Driver Carrier, F.Cu at (68.5, 63.9)
- added U3: TB67H420FTG Dual/Single Motor Driver Carrier, TB67H420FTG Dual_Single Motor Driver Carrier:TB67H420FTG DualSingle Motor Driver Carrier, F.Cu at (95.0, 63.9)
- added U4: TB67H420FTG Dual/Single Motor Driver Carrier, TB67H420FTG Dual_Single Motor Driver Carrier:TB67H420FTG DualSingle Motor Driver Carrier, F.Cu at (121.5, 63.9)
- added U5: TB67H420FTG Dual/Single Motor Driver Carrier, TB67H420FTG Dual_Single Motor Driver Carrier:TB67H420FTG DualSingle Motor Driver Carrier, F.Cu at (148.0, 63.9)
- added U7: NXV55UNR, NXV55UNR:TRANS_BC846B,215, F.Cu at (133.6, 159.5)
- added U9: DEV-16771, DEV-16771:MODULE_DEV-16771, F.Cu at (87.2, 89.3)

Commit message: abt halfway done with line 3.0
Parts:
- removed C15: 10uF, Capacitor_SMD:C_0805_2012Metric
- removed C16: 0.1uF, Capacitor_SMD:C_0805_2012Metric
- removed C17: 3.3nF, Capacitor_SMD:C_0805_2012Metric
- removed C18: 22uF, Capacitor_SMD:C_0805_2012Metric
- removed C5: 1uF, Capacitor_SMD:C_0805_2012Metric
- removed D5: STTH2002G-TR, Package_TO_SOT_SMD:TO-263-2
- removed Q2: BSC040N10NS5, Package_TO_SOT_SMD:TDSON-8-1
- removed R33: 10K, Resistor_SMD:R_0805_2012Metric
- removed U10: TPS62132, Package_DFN_QFN:VQFN-16-1EP_3x3mm_P0.5mm_EP1.68x1.68mm_ThermalVias
- removed U11: TPS62133, Package_DFN_QFN:VQFN-16-1EP_3x3mm_P0.5mm_EP1.68x1.68mm_ThermalVias
- removed U3: TB67H420FTG Dual/Single Motor Driver Carrier, TB67H420FTG Dual_Single Motor Driver Carrier:TB67H420FTG DualSingle Motor Driver Carrier
- added C11: 1uF, Capacitor_SMD:C_0805_2012Metric, F.Cu at (292.0, 205.6)
- added C12: 100uF, Capacitor_THT:CP_Radial_D10.0mm_P5.00mm, F.Cu at (166.6, 100.0)
- added C13: 560uF, Capacitor_THT:CP_Radial_D18.0mm_P7.50mm, F.Cu at (119.3, 84.5)
- added C14: 560uF, Capacitor_THT:CP_Radial_D18.0mm_P7.50mm, F.Cu at (173.3, 84.5)
- added D4: STTH2002G-TR, Package_TO_SOT_SMD:TO-263-2, F.Cu at (266.4, 148.7)
- added Q1: BSC040N10NS5, Package_TO_SOT_SMD:TDSON-8-1, F.Cu at (303.1, 167.1)
- added U6: LM2587S-ADJ, LM2587S-ADJ:VREG_TPS79625KTTR, F.Cu at (282.0, 222.0)
- added U8: TB67H420FTG Dual/Single Motor Driver Carrier, TB67H420FTG Dual_Single Motor Driver Carrier:TB67H420FTG DualSingle Motor Driver Carrier, F.Cu at (68.0, 150.0)
- A1, A10, A11, A12, A13, A14, A15, A16, A2, A3, A4, A5, A6, A7, A8, A9, LED1, LED10, LED11, LED12, LED13, LED14, LED15, LED16, LED2, LED3, LED4, LED5, LED6, LED7, LED8, LED9, R10, R12, R14, R16, R17, R19, R21, R23, R26, R28, R4, R6: moved to B.Cu
- C1: value 100uF -> 10uF; footprint Capacitor_THT:CP_Radial_D10.0mm_P5.00mm -> Capacitor_SMD:C_0805_2012Metric
- C10: value 0.1uF -> 100uF; footprint Capacitor_SMD:C_0805_2012Metric -> Capacitor_THT:CP_Radial_D10.0mm_P5.00mm
- C2: value 1uF -> 10uF
- C3, C4: value 560uF -> 0.1uF; footprint Capacitor_THT:CP_Radial_D18.0mm_P7.50mm -> Capacitor_SMD:C_0805_2012Metric
- C6: value 100uF -> 3.3nF; footprint Capacitor_THT:CP_Radial_D10.0mm_P5.00mm -> Capacitor_SMD:C_0805_2012Metric
- C7: value 22uF -> 3.3nF
- C8: value 10uF -> 22uF
- C9: value 3.3nF -> 22uF
- D1: value SS510 -> STTH2002G-TR; footprint Diode_SMD:D_SOD-128 -> Package_TO_SOT_SMD:TO-263-2
- D3: value STTH2002G-TR -> SS510; footprint Package_TO_SOT_SMD:TO-263-2 -> Diode_SMD:D_SOD-128
- J1: value Solenoid -> BATTERY POWER; footprint TerminalBlock:TerminalBlock_bornier-2_P5.08mm -> Connector_AMASS:AMASS_XT60-F_1x02_P7.20mm_Vertical
- J11: value Kicker Voltmeter -> I2C; footprint TerminalBlock:TerminalBlock_bornier-2_P5.08mm -> Connector_AMASS:AMASS_XT30U-F_1x02_P5.0mm_Vertical
- J5: value Motor 2 -> Kicker Voltmeter; footprint Connector_PinSocket_2.54mm:PinSocket_1x06_P2.54mm_Vertical -> TerminalBlock:TerminalBlock_bornier-2_P5.08mm
- J6: value Motor 4 -> Solenoid; footprint Connector_PinSocket_2.54mm:PinSocket_1x06_P2.54mm_Vertical -> TerminalBlock:TerminalBlock_bornier-2_P5.08mm
- J7: value BATTERY POWER -> Motor 2; footprint Connector_AMASS:AMASS_XT60-F_1x02_P7.20mm_Vertical -> Connector_PinSocket_2.54mm:PinSocket_1x06_P2.54mm_Vertical
- J8: value I2C TO MASTER -> Motor 4; footprint Connector_JST:JST_XH_B4B-XH-AM_1x04_P2.50mm_Vertical -> Connector_PinSocket_2.54mm:PinSocket_1x06_P2.54mm_Vertical
- L1: value 56uH -> 2.2uH
- L3: value 2.2uH -> 56uH
- R1: value 2K94 -> 12R; moved to B.Cu
- R11, R13, R15, R25, R27, R31, R9: value 12R -> 10K; moved to B.Cu
- R18, R20, R22, R24, R5, R7, R8: value 10K -> 12R; moved to B.Cu
- R2: value 57K -> 12R; moved to B.Cu
- R29: value CT6EP103 -> 10K; footprint POT_CT-6EP_NDC:POT_CT-6EP_NDC -> Resistor_SMD:R_0805_2012Metric; moved to B.Cu
- R3: value 1K5 -> 12R; moved to B.Cu
- R30, R32: value 100K -> 10K; moved to B.Cu
- R34: value 12R -> 100K
- R35: value 10K -> 100K
- R36: value 12R -> 2K94
- R37: value 10K -> 1K5
- R38: value 12R -> CT6EP103; footprint Resistor_SMD:R_0805_2012Metric -> POT_CT-6EP_NDC:POT_CT-6EP_NDC
- R39: value 10K -> 57K
- U1: value LM2587S-ADJ -> TPS62132; footprint LM2587S-ADJ:VREG_TPS79625KTTR -> Package_DFN_QFN:VQFN-16-1EP_3x3mm_P0.5mm_EP1.68x1.68mm_ThermalVias
- U2: value TB67H420FTG Dual/Single Motor Driver Carrier -> TPS62133; footprint TB67H420FTG Dual_Single Motor Driver Carrier:TB67H420FTG DualSingle Motor Driver Carrier -> Package_DFN_QFN:VQFN-16-1EP_3x3mm_P0.5mm_EP1.68x1.68mm_ThermalVias
- U7: value NXV55UNR -> TB67H420FTG Dual/Single Motor Driver Carrier; footprint NXV55UNR:TRANS_BC846B,215 -> TB67H420FTG Dual_Single Motor Driver Carrier:TB67H420FTG DualSingle Motor Driver Carrier
- moved U2 252.6 mm to (301.6, 161.1)
- moved L3 219.6 mm to (282.0, 197.6)
- moved L1 209.6 mm to (280.4, 124.8)
- moved L2 209.6 mm to (280.4, 138.9)
- moved C3 199.1 mm to (275.6, 167.5)
- moved D3 198.7 mm to (292.0, 196.6), turned to 180 degrees
- moved C4 197.6 mm to (280.1, 161.5)
- moved R37 183.8 mm to (288.0, 213.5), turned to 90 degrees
- moved C8 183.6 mm to (284.5, 161.5)
- moved C9 183.6 mm to (284.5, 164.5)
- moved R36 181.0 mm to (288.0, 205.6)
- moved C7 179.6 mm to (280.1, 167.5)
- moved R39 179.6 mm to (294.0, 201.6), turned to 90 degrees
- moved R38 178.9 mm to (288.0, 207.6)
- moved J9 178.4 mm to (161.0, 247.2), turned to 180 degrees
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Connections:
- A1 pad 2: /SEN1 -> /21
- A10 pad 2: /SEN1 -> /38
- A11 pad 2: /SEN1 -> /39
- A12 pad 2: /SEN1 -> /40
- A13 pad 2: /SEN1 -> /41
- A14 pad 2: /SEN1 -> /SEN14
- A15 pad 2: /SEN1 -> /SEN15
- A16 pad 2: /SEN1 -> /16
- A2 pad 2: /SEN1 -> /26
- A3 pad 2: /SEN1 -> /SEN3
- A4 pad 2: /SEN1 -> /23
- A5 pad 2: /SEN1 -> /20
- A6 pad 2: /SEN1 -> /27
- A7 pad 2: /SEN1 -> /SEN7
- A8 pad 2: /SEN1 -> /22
- A9 pad 2: /SEN1 -> /17
- C10 pad 1: Net-(D3-K) -> +15V
- C2 pad 1: Net-(C2-Pad1) -> Net-(D2-K)
- C2 pad 2: GND -> Net-(U2-AGND)
- C4 pad 1: Net-(D1-K) -> Net-(D2-K)
- C4 pad 2: GND -> Net-(U2-AGND)
- C6 pad 1: +15V -> GND
- C6 pad 2: GND -> Net-(U1-SS/TR)
- C7 pad 1: +3V3 -> Net-(U2-AGND)
- C7 pad 2: GND -> Net-(U2-SS/TR)
- C8 pad 1: Net-(D3-K) -> +3V3
- C9 pad 1: GND -> +5V
- C9 pad 2: Net-(U10-SS/TR) -> GND
- D1 pad 1: Net-(D1-K) -> unconnected-(D1-NC-Pad1)
- D1 pad 2: Net-(D1-A) -> Net-(D1-K)
- D2 pad 3: unconnected-(D2-A-Pad3) -> +15V
- D3 pad 1: unconnected-(D3-NC-Pad1) -> Net-(D3-K)
- D3 pad 2: Net-(D3-K) -> Net-(D3-A)
- J1 pad 1: Net-(D1-K) -> +15V
- J1 pad 2: Net-(D5-K) -> GND
- J11 pad 1: Net-(D1-K) -> /18
- J11 pad 2: GND -> /19
- J3 pad 5: /30 -> /M1ENCA
- J3 pad 6: /31 -> /M1ENCB
- J4 pad 5: /28 -> /M3ENCA
- J4 pad 6: /29 -> /M3ENCB
- J5 pad 1: Net-(J5-Pin_1) -> Net-(D3-K)
- J5 pad 2: Net-(J5-Pin_2) -> GND
- J6 pad 1: Net-(J6-Pin_1) -> Net-(D3-K)
- J6 pad 2: Net-(J6-Pin_2) -> Net-(D4-K)
- J7 pad 1: +15V -> Net-(J7-Pin_1)
- J7 pad 2: GND -> Net-(J7-Pin_2)
- J8 pad 1: /32 -> Net-(J8-Pin_1)
- J8 pad 2: /18 -> Net-(J8-Pin_2)
- J8 pad 3: /19 -> GND
- J8 pad 4: GND -> +3V3
- J9 pad 18: /14 -> /26
- J9 pad 19: /15 -> /27
- L1 pad 1: +15V -> Net-(L1-Pad1)
- L1 pad 2: Net-(D1-A) -> +3V3
- L2 pad 2: +3V3 -> +5V
- L3 pad 1: Net-(L3-Pad1) -> +15V
- L3 pad 2: +5V -> Net-(D3-A)
- LED1 pad 1: /MSFTDRN -> GND
- LED10 pad 1: /MSFTDRN -> GND
- LED11 pad 1: /MSFTDRN -> GND
- LED12 pad 1: /MSFTDRN -> GND
- LED13 pad 1: /MSFTDRN -> GND
- LED14 pad 1: /MSFTDRN -> GND
- LED15 pad 1: /MSFTDRN -> GND
- LED16 pad 1: /MSFTDRN -> GND
- LED2 pad 1: /MSFTDRN -> GND
- LED3 pad 1: /MSFTDRN -> GND
- LED4 pad 1: /MSFTDRN -> GND
- LED5 pad 1: /MSFTDRN -> GND
- LED6 pad 1: /MSFTDRN -> GND
- LED7 pad 1: /MSFTDRN -> GND
- LED8 pad 1: /MSFTDRN -> GND
- LED9 pad 1: /MSFTDRN -> GND
- R1 pad 1: Net-(U1-COMP) -> +3V3
- R1 pad 2: Net-(C2-Pad1) -> Net-(LED1-Pad2)
- R10 pad 2: /SEN1 -> /26
- R11 pad 1: +3V3 -> GND
- R11 pad 2: Net-(LED4-Pad2) -> /SEN3
- R12 pad 2: /SEN1 -> /23
- R13 pad 1: +3V3 -> GND
- R13 pad 2: Net-(LED5-Pad2) -> /20
- R14 pad 2: /SEN1 -> /27
- R15 pad 1: +3V3 -> GND
- R15 pad 2: Net-(LED6-Pad2) -> /SEN7
- R16 pad 2: /SEN1 -> /22
- R17 pad 2: Net-(LED7-Pad2) -> Net-(LED9-Pad2)
- R18 pad 1: GND -> +3V3
- R18 pad 2: /SEN1 -> Net-(LED10-Pad2)
- R19 pad 2: Net-(LED8-Pad2) -> Net-(LED11-Pad2)
- R2 pad 1: Net-(D1-K) -> +3V3
- R2 pad 2: Net-(R2-Pad2) -> Net-(LED2-Pad2)
- R20 pad 1: GND -> +3V3
- R20 pad 2: /SEN1 -> Net-(LED12-Pad2)
- R21 pad 2: Net-(LED9-Pad2) -> Net-(LED13-Pad2)
- R22 pad 1: GND -> +3V3
- R22 pad 2: /SEN1 -> Net-(LED14-Pad2)
- R23 pad 2: Net-(LED10-Pad2) -> Net-(LED15-Pad2)
- R24 pad 1: GND -> +3V3
- R24 pad 2: /SEN1 -> Net-(LED16-Pad2)
- R25 pad 1: +3V3 -> GND
- R25 pad 2: Net-(LED11-Pad2) -> /17
- R26 pad 2: /SEN1 -> /38
- R27 pad 1: +3V3 -> GND
- R27 pad 2: Net-(LED12-Pad2) -> /39
- R28 pad 2: /SEN1 -> /40
- R29 pad 1: Net-(U1-FB) -> GND
- R29 pad 2: Net-(U1-FB) -> /41
- R3 pad 1: Net-(U1-FB) -> +3V3
- R3 pad 2: GND -> Net-(LED3-Pad2)
- R30 pad 1: Net-(U10-PG) -> GND
- R30 pad 2: +3V3 -> /SEN14
- R31 pad 1: +3V3 -> GND
- R31 pad 2: Net-(LED13-Pad2) -> /SEN15
- R32 pad 1: Net-(U11-PG) -> GND
- R32 pad 2: +5V -> /16
- R34 pad 1: +3V3 -> Net-(U1-PG)
- R34 pad 2: Net-(LED14-Pad2) -> +3V3
- R35 pad 1: GND -> Net-(U2-PG)
- R35 pad 2: /SEN1 -> +5V
- R36 pad 1: +3V3 -> Net-(U6-COMP)
- R36 pad 2: Net-(LED15-Pad2) -> Net-(C11-Pad1)
- R37 pad 1: GND -> Net-(U6-FB)
- R37 pad 2: /SEN1 -> GND
- R38 pad 1: +3V3 -> Net-(U6-FB)
- R38 pad 2: Net-(LED16-Pad2) -> Net-(U6-FB)
- R39 pad 1: GND -> Net-(D3-K)
- R39 pad 2: /SEN1 -> Net-(R38-Pad3)
- R4 pad 2: Net-(LED1-Pad2) -> Net-(LED4-Pad2)
- R5 pad 1: GND -> +3V3
- R5 pad 2: /SEN1 -> Net-(LED5-Pad2)
- R6 pad 2: Net-(LED2-Pad2) -> Net-(LED6-Pad2)
- R7 pad 1: GND -> +3V3
- R7 pad 2: /2 -> Net-(LED7-Pad2)
- R8 pad 1: GND -> +3V3
- R8 pad 2: /SEN1 -> Net-(LED8-Pad2)
- R9 pad 1: +3V3 -> GND
- R9 pad 2: Net-(LED3-Pad2) -> /21
- U1 pad 1: Net-(U1-COMP) -> Net-(L1-Pad1)
- U1 pad 2: Net-(U1-FB) -> Net-(L1-Pad1)
- U1 pad 3: GND -> Net-(L1-Pad1)
- U1 pad 4: Net-(D1-A) -> Net-(U1-PG)
- U1 pad 5: +15V -> GND
- U2 pad 1: unconnected-(U2-VM-Pad1) -> Net-(L2-Pad1)
- U2 pad 10: unconnected-(U2-LO1-Pad10) -> Net-(D2-K)
- U2 pad 11: unconnected-(U2-LO2-Pad11) -> Net-(D2-K)
- U2 pad 12: unconnected-(U2-VREFA-Pad12) -> Net-(D2-K)
- U2 pad 13: unconnected-(U2-VREFB-Pad13) -> Net-(D2-K)
- U2 pad 14: +15V -> +5V
- U2 pad 16: Net-(J4-Pin_1) -> GND
- U2 pad 17: Net-(J4-Pin_1) -> GND
- U2 pad 2: GND -> Net-(L2-Pad1)
- U2 pad 3: unconnected-(U2-VCC-Pad3) -> Net-(L2-Pad1)
- U2 pad 4: /41 -> Net-(U2-PG)
- U2 pad 5: /40 -> GND
- U2 pad 6: /5 -> Net-(U2-AGND)
- U2 pad 7: unconnected-(U2-INB1-Pad7) -> Net-(U2-AGND)
- U2 pad 8: unconnected-(U2-INB2-Pad8) -> Net-(U2-AGND)
- U2 pad 9: unconnected-(U2-PWMB-Pad9) -> Net-(U2-SS/TR)
- U4 pad 16: Net-(J5-Pin_1) -> Net-(J3-Pin_1)
- U4 pad 17: Net-(J5-Pin_1) -> Net-(J3-Pin_1)
- U4 pad 18: Net-(J5-Pin_2) -> Net-(J3-Pin_2)
- U4 pad 19: Net-(J5-Pin_2) -> Net-(J3-Pin_2)
- U4 pad 4: /10 -> /M1IN1
- U4 pad 5: /33 -> /M1IN2
- U4 pad 6: /4 -> /M1PWM
- U5 pad 16: Net-(J6-Pin_1) -> Net-(J4-Pin_1)
- U5 pad 17: Net-(J6-Pin_1) -> Net-(J4-Pin_1)
- U5 pad 18: Net-(J6-Pin_2) -> Net-(J4-Pin_2)
- U5 pad 19: Net-(J6-Pin_2) -> Net-(J4-Pin_2)
- U5 pad 4: /39 -> /M3IN1
- U5 pad 5: /38 -> /M3IN2
- U5 pad 6: /6 -> /M3PWM
- U7 pad 1: /2 -> unconnected-(U7-VM-Pad1)
- U7 pad 3: /MSFTDRN -> unconnected-(U7-VCC-Pad3)
- U9 pad 26: /14 -> /26
- U9 pad 27: /15 -> /27
Routing:
- net /21: track 0.00 -> 190.0 mm
- net /20: track 0.00 -> 155.6 mm
- net /23: track 0.00 -> 127.3 mm
- net /17: track 0.00 -> 122.5 mm
- net /26: track 0.00 -> 107.5 mm
- net /22: track 0.00 -> 105.8 mm
- net /16: track 0.00 -> 99.9 mm
- net /38: track 0.00 -> 91.0 mm
- net /39: track 0.00 -> 81.7 mm
- net /SEN15: track 0.00 -> 76.6 mm
- net /27: track 0.00 -> 76.6 mm
- net Net-(J3-Pin_1): track 0.00 -> 71.7 mm
- net /40: track 0.00 -> 67.6 mm
- net +3V3: track 0.00 -> 65.8 mm
- net /SEN14: track 0.00 -> 63.1 mm
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- added copper zone on B.Cu, net GND
- added copper zone on F.Cu, net GND
Other:
- board outline added: 206 x 197.4 mm

Commit message: Line 3.0 save
Connections:
- A3 pad 2: /SEN3 -> /24
- A7 pad 2: /SEN7 -> /25
- R11 pad 2: /SEN3 -> /24
- R15 pad 2: /SEN7 -> /25
Routing:
- net /24: track 3.42 -> 27.8 mm
- net /25: track 3.42 -> 17.7 mm
- net /SEN7: track 4.11 -> 0.00 mm
- net /SEN3: track 4.11 -> 0.00 mm

Commit message: CLEAN UP 3.0 LINE SCH
Parts:
- added REF**: gv2 3d outline, gv2outlineforkicad:gv2 3d outline, F.Cu at (150.0, 150.0)
- moved J6 156.8 mm to (144.5, 110.0)
- moved R34 154.3 mm to (159.7, 180.2), turned to 90 degrees
- moved U1 147.4 mm to (156.4, 180.6)
- moved R35 145.8 mm to (179.8, 202.6), turned to 180 degrees
- moved D1 133.4 mm to (143.5, 175.9), turned to -90 degrees
- moved L1 132.9 mm to (156.0, 171.5), turned to 90 degrees
- moved C6 129.3 mm to (152.2, 183.8)
- moved U2 129.1 mm to (180.5, 205.9), turned to 90 degrees
- moved L2 128.1 mm to (171.4, 206.2), turned to 180 degrees
- moved C1 124.6 mm to (152.2, 179.2), turned to 180 degrees
- moved C8 124.3 mm to (161.7, 180.2), turned to -90 degrees
- moved C3 124.2 mm to (152.2, 181.5), turned to 180 degrees
- moved D2 122.5 mm to (175.8, 218.8)
- moved C9 110.8 mm to (179.8, 200.6)
- moved C4 110.0 mm to (181.4, 210.0), turned to -90 degrees
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Connections:
- A14 pad 2: /SEN14 -> /14
- A15 pad 2: /SEN15 -> /15
- C2 pad 2: Net-(U2-AGND) -> GND
- C4 pad 2: Net-(U2-AGND) -> GND
- C7 pad 1: Net-(U2-AGND) -> GND
- R30 pad 2: /SEN14 -> /14
- R31 pad 2: /SEN15 -> /15
- U2 pad 6: Net-(U2-AGND) -> GND
- U2 pad 7: Net-(U2-AGND) -> GND
- U2 pad 8: Net-(U2-AGND) -> GND
Routing:
- net +15V: track 0.00 -> 459.8 mm
- net /SEN15: track 76.6 -> 0.00 mm
- net /15: track 3.42 -> 80.0 mm
- net /SEN14: track 63.1 -> 0.00 mm
- net /14: track 3.42 -> 66.5 mm
- net Net-(J8-Pin_1): track 0.00 -> 60.9 mm
- net Net-(J8-Pin_2): track 0.00 -> 57.1 mm
- net Net-(J7-Pin_1): track 0.00 -> 47.0 mm
- net Net-(J7-Pin_2): track 0.00 -> 35.4 mm
- net Net-(D2-K): track 0.00 -> 34.5 mm
- net GND: track 0.00 -> 33.6 mm
- net Net-(D1-K): track 0.00 -> 32.1 mm
- net +3V3: track 65.8 -> 94.6 mm, vias 0 -> 8
- net +5V: track 18.2 -> 39.4 mm
- net Net-(U2-PG): track 0.00 -> 12.2 mm, vias 0 -> 2
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- added copper zone on F.Cu, net +3V3

Commit message: line 3.0 - good for the night
Parts:
- removed C1, C2: 10uF, Capacitor_SMD:C_0805_2012Metric
- removed C10, C12: 100uF, Capacitor_THT:CP_Radial_D10.0mm_P5.00mm
- removed C11: 1uF, Capacitor_SMD:C_0805_2012Metric
- removed C13, C14: 560uF, Capacitor_THT:CP_Radial_D18.0mm_P7.50mm
- removed C3, C4: 0.1uF, Capacitor_SMD:C_0805_2012Metric
- removed C6, C7: 3.3nF, Capacitor_SMD:C_0805_2012Metric
- removed C8, C9: 22uF, Capacitor_SMD:C_0805_2012Metric
- removed D1, D2, D4: STTH2002G-TR, Package_TO_SOT_SMD:TO-263-2
- removed D3: SS510, Diode_SMD:D_SOD-128
- removed J5: Kicker Voltmeter, TerminalBlock:TerminalBlock_bornier-2_P5.08mm
- removed J6: Solenoid, TerminalBlock:TerminalBlock_bornier-2_P5.08mm
- removed L1, L2: 2.2uH, Inductor_SMD:L_Bourns_SRR1260
- removed L3: 56uH, Inductor_SMD:L_Bourns_SRR1260
- removed Q1: BSC040N10NS5, Package_TO_SOT_SMD:TDSON-8-1
- removed R34, R35: 100K, Resistor_SMD:R_0805_2012Metric
- removed R36: 2K94, Resistor_SMD:R_0805_2012Metric
- removed R37: 1K5, Resistor_SMD:R_0805_2012Metric
- removed R38: CT6EP103, POT_CT-6EP_NDC:POT_CT-6EP_NDC
- removed R39: 57K, Resistor_SMD:R_0805_2012Metric
- removed U1: TPS62132, Package_DFN_QFN:VQFN-16-1EP_3x3mm_P0.5mm_EP1.68x1.68mm_ThermalVias
- removed U2: TPS62133, Package_DFN_QFN:VQFN-16-1EP_3x3mm_P0.5mm_EP1.68x1.68mm_ThermalVias
- removed U9: DEV-16771, DEV-16771:MODULE_DEV-16771
- added J12: RIGHT HEADERS, Connector_PinHeader_2.54mm:PinHeader_1x24_P2.54mm_Vertical, F.Cu at (139.0, 246.5)
- added J2: BACKUP 5V, Connector_AMASS:AMASS_XT30U-F_1x02_P5.0mm_Vertical, F.Cu at (235.0, 127.5)
- J10: value RIGHT HEADERS -> Motor 4; footprint Connector_PinHeader_2.54mm:PinHeader_1x24_P2.54mm_Vertical -> Connector_PinSocket_2.54mm:PinSocket_1x06_P2.54mm_Vertical
- J11: value I2C -> LEFT HEADERS; footprint Connector_AMASS:AMASS_XT30U-F_1x02_P5.0mm_Vertical -> Connector_PinHeader_2.54mm:PinHeader_1x24_P2.54mm_Vertical
- J3: value Motor 1 -> BACKUP 3V3; footprint Connector_PinSocket_2.54mm:PinSocket_1x06_P2.54mm_Vertical -> Connector_AMASS:AMASS_XT30U-F_1x02_P5.0mm_Vertical
- J4: value Motor 3 -> I2C; footprint Connector_PinSocket_2.54mm:PinSocket_1x06_P2.54mm_Vertical -> Connector_AMASS:AMASS_XT30U-F_1x02_P5.0mm_Vertical
- J7: value Motor 2 -> Motor 1
- J8: value Motor 4 -> Motor 2
- J9: value LEFT HEADERS -> Motor 3; footprint Connector_PinHeader_2.54mm:PinHeader_1x24_P2.54mm_Vertical -> Connector_PinSocket_2.54mm:PinSocket_1x06_P2.54mm_Vertical
- U6: value LM2587S-ADJ -> TB67H420FTG Dual/Single Motor Driver Carrier; footprint LM2587S-ADJ:VREG_TPS79625KTTR -> TB67H420FTG Dual_Single Motor Driver Carrier:TB67H420FTG DualSingle Motor Driver Carrier
- U8: value TB67H420FTG Dual/Single Motor Driver Carrier -> DEV-16771; footprint TB67H420FTG Dual_Single Motor Driver Carrier:TB67H420FTG DualSingle Motor Driver Carrier -> DEV-16771:MODULE_DEV-16771
- moved U6 179.6 mm to (100.0, 150.0), turned to 0 degrees
- moved J1 149.9 mm to (62.5, 127.5), turned to 0 degrees
- moved J10 133.9 mm to (95.5, 120.5), turned to 45 degrees
- moved J4 130.6 mm to (65.0, 172.5), turned to 0 degrees
- moved J8 111.8 mm to (204.5, 179.5)
- moved J7 111.8 mm to (204.5, 120.5), turned to -45 degrees
- moved U8 106.0 mm to (150.0, 217.2), turned to 90 degrees
- moved J9 94.2 mm to (95.5, 179.5), turned to 135 degrees
- moved J3 58.4 mm to (235.0, 172.5), turned to 180 degrees
- moved J11 36.5 mm to (161.0, 246.5), turned to 180 degrees
- moved U7 28.0 mm to (70.0, 150.0), turned to 0 degrees
- moved U4 2.00 mm to (230.0, 150.0)
- moved U5 2.00 mm to (200.0, 150.0)
Connections:
- J1 pad 1: +15V -> GND
- J1 pad 2: GND -> +15V
- J10 pad 1: +5V -> Net-(J10-Pin_1)
- J10 pad 2: GND -> Net-(J10-Pin_2)
- J10 pad 3: +3V3 -> GND
- J10 pad 4: /23 -> +3V3
- J10 pad 5: /22 -> /3
- J10 pad 6: /21 -> /4
- J11 pad 1: /18 -> GND
- J11 pad 2: /19 -> /0
- J3 pad 1: Net-(J3-Pin_1) -> GND
- J3 pad 2: Net-(J3-Pin_2) -> +3V3
- J4 pad 1: Net-(J4-Pin_1) -> /19
- J4 pad 2: Net-(J4-Pin_2) -> /18
- J7 pad 5: /M2ENCA -> /7
- J7 pad 6: /M2ENCB -> /8
- J8 pad 5: /M4ENCA -> /34
- J8 pad 6: /M4ENCB -> /35
- J9 pad 1: GND -> Net-(J9-Pin_1)
- J9 pad 2: /0 -> Net-(J9-Pin_2)
- J9 pad 3: /1 -> GND
- J9 pad 4: /2 -> +3V3
- J9 pad 5: /3 -> /30
- J9 pad 6: /4 -> /31
- U4 pad 16: Net-(J3-Pin_1) -> Net-(J7-Pin_1)
- U4 pad 17: Net-(J3-Pin_1) -> Net-(J7-Pin_1)
- U4 pad 18: Net-(J3-Pin_2) -> Net-(J7-Pin_2)
- U4 pad 19: Net-(J3-Pin_2) -> Net-(J7-Pin_2)
- U4 pad 4: /M1IN1 -> /2
- U4 pad 5: /M1IN2 -> /6
- U4 pad 6: /M1PWM -> /28
- U5 pad 16: Net-(J4-Pin_1) -> Net-(J8-Pin_1)
- U5 pad 17: Net-(J4-Pin_1) -> Net-(J8-Pin_1)
- U5 pad 18: Net-(J4-Pin_2) -> Net-(J8-Pin_2)
- U5 pad 19: Net-(J4-Pin_2) -> Net-(J8-Pin_2)
- U5 pad 4: /M3IN1 -> /9
- U5 pad 5: /M3IN2 -> /32
- U5 pad 6: /M3PWM -> /29
- U6 pad 1: Net-(U6-COMP) -> unconnected-(U6-VM-Pad1)
- U6 pad 2: Net-(U6-FB) -> GND
- U6 pad 3: GND -> unconnected-(U6-VCC-Pad3)
- U6 pad 4: Net-(D3-A) -> /10
- U6 pad 5: +15V -> /12
- U6 pad 6: GND -> /37
- U7 pad 16: Net-(J7-Pin_1) -> Net-(J10-Pin_1)
- U7 pad 17: Net-(J7-Pin_1) -> Net-(J10-Pin_1)
- U7 pad 18: Net-(J7-Pin_2) -> Net-(J10-Pin_2)
- U7 pad 19: Net-(J7-Pin_2) -> Net-(J10-Pin_2)
- U7 pad 4: /M2IN1 -> /11
- U7 pad 5: /M2IN2 -> /33
- U7 pad 6: /M2PWM -> /36
- U8 pad 1: unconnected-(U8-VM-Pad1) -> /1
- U8 pad 10: unconnected-(U8-LO1-Pad10) -> /10
- U8 pad 11: unconnected-(U8-LO2-Pad11) -> /11
- U8 pad 12: unconnected-(U8-VREFA-Pad12) -> /12
- U8 pad 13: unconnected-(U8-VREFB-Pad13) -> /13
- U8 pad 14: +15V -> /14
- U8 pad 15: GND -> /15
- U8 pad 16: Net-(J8-Pin_1) -> /16
- U8 pad 17: Net-(J8-Pin_1) -> /17
- U8 pad 18: Net-(J8-Pin_2) -> /18
- U8 pad 19: Net-(J8-Pin_2) -> /19
- U8 pad 2: GND -> /2
- U8 pad 20: Net-(U8-HBMODE) -> /20
- U8 pad 21: Net-(U8-HBMODE) -> /21
- U8 pad 22: unconnected-(U8-TBLKAB-Pad22) -> /22
- U8 pad 23: Net-(U8-HBMODE) -> /23
- U8 pad 3: unconnected-(U8-VCC-Pad3) -> /3
- U8 pad 4: /M4IN1 -> /4
- U8 pad 5: /M4IN2 -> /5
- U8 pad 6: /M4PWM -> /6
- U8 pad 7: unconnected-(U8-INB1-Pad7) -> /7
- U8 pad 8: unconnected-(U8-INB2-Pad8) -> /8
- U8 pad 9: unconnected-(U8-PWMB-Pad9) -> /9
Routing:
- net +15V: track 459.8 -> 0.00 mm
- net +3V3: track 94.6 -> 418.5 mm, vias 8 -> 18
- net /19: track 17.0 -> 103.0 mm, vias 0 -> 1
- net /18: track 16.0 -> 99.1 mm, vias 0 -> 1
- net /15: track 80.0 -> 7.49 mm
- net Net-(J3-Pin_1): track 71.7 -> 0.00 mm
- net Net-(J3-Pin_2): track 59.5 -> 0.00 mm
- net Net-(J10-Pin_2): track 0.00 -> 41.3 mm
- net +5V: track 39.4 -> 0.00 mm
- net Net-(J9-Pin_1): track 0.00 -> 38.5 mm
- net Net-(J10-Pin_1): track 0.00 -> 36.7 mm
- net Net-(D2-K): track 34.5 -> 0.00 mm
- net GND: track 33.6 -> 0.00 mm
- net Net-(J4-Pin_1): track 32.2 -> 0.00 mm
- net Net-(D1-K): track 32.1 -> 0.00 mm
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- added copper zone on F.Cu, net +15V
- removed copper zone on F.Cu, net +3V3
- removed copper zone on F.Cu, net GND
Other:
- outline, holes or cut-outs redrawn
