File: Goku _ Vegeta/3.0/Line 3.0 - GV3/Line 3.0.kicad_pcb (KiCad board)
At the start: 2 copper layers, 206 x 197.4 mm, 80 parts, among them J1 BATTERY POWER, J10 Motor 4, J11 LEFT HEADERS, J12 RIGHT HEADERS, J2 BACKUP 5V, J3 BACKUP 3V3, J4 I2C, J7 Motor 1, J8 Motor 2, J9 Motor 3, U4 TB67H420FTG Dual/Single Motor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, U5 TB67H420FTG Dual/Single Motor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, U6 TB67H420FTG Dual/Single Motor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, U7 TB67H420FTG Dual/Single Motor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, U8 DEV-16771

Commit message: LINE 3.0 - teensy - M driver routing +  added teensy programming. + on off switch breakout
Parts:
- removed REF**: gv2 3d outline, gv2outlineforkicad:gv2 3d outline
- added C1: 10uF, Capacitor_SMD:C_0805_2012Metric, F.Cu at (21.8, 43.2)
- added C10: 1uF, Capacitor_SMD:C_0805_2012Metric, F.Cu at (30.7, 49.2)
- added C11: 100uF, Capacitor_THT:CP_Radial_D10.0mm_P5.00mm, F.Cu at (37.2, 53.9)
- added C12: 560uF, Capacitor_THT:CP_Radial_D18.0mm_P7.50mm, F.Cu at (6.07, 9.28)
- added C13: 560uF, Capacitor_THT:CP_Radial_D18.0mm_P7.50mm, F.Cu at (6.07, 28.8)
- added C2: 10uF, Capacitor_SMD:C_0805_2012Metric, F.Cu at (21.8, 46.2)
- added C3: 0.1uF, Capacitor_SMD:C_0805_2012Metric, F.Cu at (21.8, 49.2)
- added C4: 0.1uF, Capacitor_SMD:C_0805_2012Metric, F.Cu at (26.3, 43.2)
- added C5: 3.3nF, Capacitor_SMD:C_0805_2012Metric, F.Cu at (26.3, 46.2)
- added C6: 3.3nF, Capacitor_SMD:C_0805_2012Metric, F.Cu at (26.3, 49.2)
- added C7: 22uF, Capacitor_SMD:C_0805_2012Metric, F.Cu at (30.7, 43.2)
- added C8: 22uF, Capacitor_SMD:C_0805_2012Metric, F.Cu at (30.7, 46.2)
- added C9: 100uF, Capacitor_THT:CP_Radial_D10.0mm_P5.00mm, F.Cu at (37.2, 42.3)
- added D1: STTH2002G-TR, Package_TO_SOT_SMD:TO-263-2, F.Cu at (44.4, 5.67)
- added D2: STTH2002G-TR, Package_TO_SOT_SMD:TO-263-2, F.Cu at (44.4, 18.0)
- added D3: SS510, Diode_SMD:D_SOD-128, F.Cu at (14.8, 55.4)
- added D4: STTH2002G-TR, Package_TO_SOT_SMD:TO-263-2, F.Cu at (44.4, 30.4)
- added J13: MID HEADERS, Connector_PinHeader_2.54mm:PinHeader_1x05_P2.54mm_Vertical, F.Cu at (144.9, 185.2)
- added J5: Kicker Voltmeter, TerminalBlock:TerminalBlock_bornier-2_P5.08mm, F.Cu at (2.73, 43.1)
- added J6: Solenoid, TerminalBlock:TerminalBlock_bornier-2_P5.08mm, F.Cu at (2.73, 52.2)
- added L1: 2.2uH, Inductor_SMD:L_Bourns_SRR1260, F.Cu at (26.6, 6.53)
- added L2: 2.2uH, Inductor_SMD:L_Bourns_SRR1260, F.Cu at (26.6, 20.6)
- added L3: 56uH, Inductor_SMD:L_Bourns_SRR1260, F.Cu at (26.6, 34.6)
- added Q1: BSC040N10NS5, Package_TO_SOT_SMD:TDSON-8-1, F.Cu at (23.7, 54.0)
- added R33: 100K, Resistor_SMD:R_0805_2012Metric, F.Cu at (13.3, 40.1)
- added R34: 100K, Resistor_SMD:R_0805_2012Metric, F.Cu at (13.3, 43.0)
- added R35: 2K94, Resistor_SMD:R_0805_2012Metric, F.Cu at (13.3, 46.0)
- added R36: 1K5, Resistor_SMD:R_0805_2012Metric, F.Cu at (13.3, 48.9)
- added R38: 57K, Resistor_SMD:R_0805_2012Metric, F.Cu at (13.3, 51.9)
- added U1: TPS62132, Package_DFN_QFN:VQFN-16-1EP_3x3mm_P0.5mm_EP1.68x1.68mm_ThermalVias, F.Cu at (48.1, 39.2)
- added U2: TPS62133, Package_DFN_QFN:VQFN-16-1EP_3x3mm_P0.5mm_EP1.68x1.68mm_ThermalVias, F.Cu at (48.1, 44.5)
- added U3: LM2587S-ADJ, LM2587S-ADJ:VREG_TPS79625KTTR, F.Cu at (26.5, 68.2)
- moved J11 0.76 mm to (161.0, 247.2)
- moved J12 0.76 mm to (139.0, 247.2)
- moved U8 0.76 mm to (150.0, 218.0)
Connections:
- J10 pad 5: /3 -> /29
- J10 pad 6: /4 -> /28
- J7 pad 5: /7 -> /5
- J7 pad 6: /8 -> /6
- J8 pad 5: /34 -> /7
- J8 pad 6: /35 -> /8
- J9 pad 5: /30 -> /34
- J9 pad 6: /31 -> /33
- U4 pad 4: /2 -> /4
- U4 pad 5: /6 -> /3
- U4 pad 6: /28 -> /2
- U5 pad 4: /9 -> /11
- U5 pad 5: /32 -> /10
- U5 pad 6: /29 -> /9
- U6 pad 4: /10 -> /30
- U6 pad 5: /12 -> /31
- U6 pad 6: /37 -> /32
- U7 pad 4: /11 -> /35
- U7 pad 5: /33 -> /36
- U7 pad 6: /36 -> /37
- U8 pad ON/OFF: unconnected-(U8-PadON/OFF) -> /ON/OFF
- U8 pad PROGRAM: unconnected-(U8-PadPROGRAM) -> /PROGRAM
Routing:
- net /5: track 3.38 -> 140.0 mm
- net /6: track 3.38 -> 136.6 mm
- net /2: track 3.38 -> 122.0 mm
- net /3: track 3.38 -> 121.7 mm
- net /30: track 3.38 -> 121.3 mm
- net /4: track 3.38 -> 117.3 mm
- net /31: track 3.38 -> 117.0 mm
- net /28: track 3.38 -> 112.0 mm
- net /29: track 3.38 -> 112.0 mm
- net /32: track 3.38 -> 108.5 mm
- net /35: track 3.38 -> 105.1 mm
- net /37: track 3.38 -> 104.6 mm
- net /36: track 3.38 -> 104.6 mm
- net /9: track 3.38 -> 87.2 mm
- net /11: track 3.38 -> 87.1 mm
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Other:
- board text added: "NOTE: ALL TEENSY 4.1 3V3 LINES ARE NOT CONNECTED"
