File: Goku _ Vegeta/3.0/Main 3.0 - GV3/Main 3.0.kicad_pcb (KiCad board)
At the start: 2 copper layers, 215 x 206.6 mm, 43 parts, among them J1 JST-XH M1 ENC, J10 Conn_01x08_Female, J11 Motor Driver Inputs, J12 OpenMV H7, J13 JST-XH Screen, J14 Conn_01x08_Female, J15 691137710002, J16 691137710002, J17 Conn_01x08_Female, J18 Conn_01x18_Female, J19 Conn_01x10_Female, J2 JST-XH M2 ENC, J20 Conn_01x08_Female, J21 Conn_01x08_Female, J22 Conn_01x18_Female, J23 Line PCB 2, J24 B3B-XH-A(LF)(SN), J25 B2B-XH-A(LF)(SN), J3 JST-XH M3 ENC, J4 JST-XH M4 ENC, J5 XT60-M, J6 691137710002, J7 XT60-M, J8 XT60-M, J9 Line PCB 1, U1 DC-DC_Buck_Converter_7-24V_to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, U4 Adafruit_BNO055_STEMMA_QT

Commit message: move to 3.1
Parts:
- removed A1: A000067, A000067:ARDUINO_A000067_FLIPPED
- removed C3, C4: 10UF, Capacitor_SMD:C_0805_2012Metric
- removed J24: B3B-XH-A(LF)(SN), B3B-XH-A_LF__SN_:JST_B3B-XH-A(LF)(SN)
- removed J25: B2B-XH-A(LF)(SN), B2B-XH-A_LF__SN_:JST_B2B-XH-A(LF)(SN)
- removed R13, R14: 10K, Resistor_SMD:R_0805_2012Metric
- removed TP1: TestPoint - 5V, TestPoint:TestPoint_THTPad_D2.0mm_Drill1.0mm
- removed TP18: LOGIC_SWITCH, TestPoint:TestPoint_THTPad_D2.0mm_Drill1.0mm
- removed TP2: TestPoint - SCL, TestPoint:TestPoint_THTPad_D2.0mm_Drill1.0mm
- removed TP3: TestPoint - SDA, TestPoint:TestPoint_THTPad_D2.0mm_Drill1.0mm
- removed TP4: TestPoint - TX, TestPoint:TestPoint_THTPad_D2.0mm_Drill1.0mm
- removed TP5: TestPoint - RX, TestPoint:TestPoint_THTPad_D2.0mm_Drill1.0mm
- removed TP6: TestPoint - GND, TestPoint:TestPoint_THTPad_D2.0mm_Drill1.0mm
- added C2: 100uF, Capacitor_THT:CP_Radial_D10.0mm_P5.00mm, F.Cu at (502.9, 152.9)
- added D1: LED, 5mm Pitch 2-Pin Screw Terminal Block:5mm Pitch 2-Pin Screw Terminal Block, F.Cu at (493.6, 139.8)
- added Q1: Q_Photo_NPN, 5mm Pitch 2-Pin Screw Terminal Block:5mm Pitch 2-Pin Screw Terminal Block, F.Cu at (493.6, 158.1)
- added R1: 10K, Resistor_SMD:R_0805_2012Metric, F.Cu at (501.6, 160.1)
- added R10: 10K, Resistor_SMD:R_0805_2012Metric, F.Cu at (510.4, 163.1)
- added R11: 10K, Resistor_SMD:R_0805_2012Metric, F.Cu at (510.4, 166.0)
- added R12: 10K, Resistor_SMD:R_0805_2012Metric, F.Cu at (510.4, 169.0)
- added R2: 10K, Resistor_SMD:R_0805_2012Metric, F.Cu at (501.6, 163.1)
- added R3: 10K, Resistor_SMD:R_0805_2012Metric, F.Cu at (501.6, 166.0)
- added R4: 10K, Resistor_SMD:R_0805_2012Metric, F.Cu at (501.6, 169.0)
- added R5: 95R, Resistor_SMD:R_0805_2012Metric, F.Cu at (506.0, 160.1)
- added R6: 10K, Resistor_SMD:R_0805_2012Metric, F.Cu at (506.0, 163.1)
- added R7: 10K, Resistor_SMD:R_0805_2012Metric, F.Cu at (506.0, 166.0)
- added R8: 10K, Resistor_SMD:R_0805_2012Metric, F.Cu at (506.0, 169.0)
- added R9: 10K, Resistor_SMD:R_0805_2012Metric, F.Cu at (510.4, 160.1)
- added REF**: GV3 Main, Main GV3:GV3 Main, F.Cu at (150.0, 150.0)
- added U2: ~, Converter_DCDC:DC-DC Multi-output Buck Converter, F.Cu at (116.9, 198.5)
- added U3: Adafruit_BNO055_STEMMA_QT, 2.3 PCBs:Adafruit IMU BNO055, F.Cu at (173.5, 212.0)
- C1: value 10UF -> 100uF; footprint Capacitor_SMD:C_0805_2012Metric -> Capacitor_THT:CP_Radial_D10.0mm_P5.00mm
- J1: value JST-XH M1 ENC -> 4S Battery; footprint B4B-XH-A_LF__SN_:JST_B4B-XH-A(LF)(SN) -> Connector_AMASS:AMASS_XT60-M_1x02_P7.20mm_Vertical
- J10: value Conn_01x08_Female -> BACKUP 3V3; footprint Connector_PinHeader_2.54mm:PinHeader_1x08_P2.54mm_Vertical -> Connector_AMASS:AMASS_XT30U-F_1x02_P5.0mm_Vertical
- J11: value Motor Driver Inputs -> I2C; footprint Box IDC header 2x5:Box IDC header 2x5 -> Connector_AMASS:AMASS_XT30U-F_1x02_P5.0mm_Vertical
- J12: value OpenMV H7 -> SPI; footprint Box IDC header 2x3:Box IDC header 2x3 -> Connector_PinSocket_2.54mm:PinSocket_1x05_P2.54mm_Vertical
- J13: value JST-XH Screen -> UART; footprint B4B-XH-A_LF__SN_:JST_B4B-XH-A(LF)(SN) -> Connector_PinSocket_2.54mm:PinSocket_1x03_P2.54mm_Vertical
- J14: value Conn_01x08_Female -> I2C; footprint Connector_PinHeader_2.54mm:PinHeader_1x08_P2.54mm_Vertical -> Connector_PinSocket_2.54mm:PinSocket_1x04_P2.54mm_Vertical
- J15, J16: value 691137710002 -> Conn_01x02_Male; footprint 5mm Pitch 2-Pin Screw Terminal Block:5mm Pitch 2-Pin Screw Terminal Block -> Connector_JST:JST_XH_B2B-XH-A_1x02_P2.50mm_Vertical
- J17, J20: value Conn_01x08_Female -> Conn_01x02_Male; footprint Connector_PinHeader_2.54mm:PinHeader_1x08_P2.54mm_Vertical -> Connector_JST:JST_XH_B2B-XH-A_1x02_P2.50mm_Vertical
- J18: value Conn_01x18_Female -> Conn_01x02_Male; footprint Connector_PinHeader_2.54mm:PinHeader_1x18_P2.54mm_Vertical -> Connector_JST:JST_XH_B2B-XH-A_1x02_P2.50mm_Vertical
- J19: value Conn_01x10_Female -> Conn_01x02_Male; footprint Connector_PinHeader_2.54mm:PinHeader_1x10_P2.54mm_Vertical -> Connector_JST:JST_XH_B2B-XH-A_1x02_P2.50mm_Vertical
- J2: value JST-XH M2 ENC -> Power Switch; footprint B4B-XH-A_LF__SN_:JST_B4B-XH-A(LF)(SN) -> Connector_AMASS:AMASS_XT30UPB-F_1x02_P5.0mm_Vertical
- J21: value Conn_01x08_Female -> LEFT HEADERS; footprint Connector_PinHeader_2.54mm:PinHeader_1x08_P2.54mm_Vertical -> Connector_PinHeader_2.54mm:PinHeader_1x24_P2.54mm_Vertical
- J22: value Conn_01x18_Female -> MID HEADERS; footprint Connector_PinHeader_2.54mm:PinHeader_1x18_P2.54mm_Vertical -> Connector_PinHeader_2.54mm:PinHeader_1x05_P2.54mm_Vertical
- J23: value Line PCB 2 -> RIGHT HEADERS; footprint Box IDC header 2x3:Box IDC header 2x3 -> Connector_PinHeader_2.54mm:PinHeader_1x24_P2.54mm_Vertical
- J3: value JST-XH M3 ENC -> 691137710002; footprint B4B-XH-A_LF__SN_:JST_B4B-XH-A(LF)(SN) -> 5mm Pitch 2-Pin Screw Terminal Block:5mm Pitch 2-Pin Screw Terminal Block
- J4: value JST-XH M4 ENC -> Battery Buzzer 1; footprint B4B-XH-A_LF__SN_:JST_B4B-XH-A(LF)(SN) -> Connector_PinSocket_2.54mm:PinSocket_1x08_P2.54mm_Vertical
- J5: value XT60-M -> Battery Buzzer 2; footprint XT60-M:XT60-M -> Connector_PinSocket_2.54mm:PinSocket_1x08_P2.54mm_Vertical
- J6: value 691137710002 -> Battery Balance 1; footprint 5mm Pitch 2-Pin Screw Terminal Block:5mm Pitch 2-Pin Screw Terminal Block -> Connector_JST:JST_XH_B3B-XH-A_1x03_P2.50mm_Vertical
- J7: value XT60-M -> Battery Balance 2; footprint XT60-M:XT60-M -> Connector_JST:JST_XH_B3B-XH-A_1x03_P2.50mm_Vertical
- J8: value XT60-M -> BATTERY POWER; footprint XT60-M:XT60-M -> Connector_AMASS:AMASS_XT30U-F_1x02_P5.0mm_Vertical
- J9: value Line PCB 1 -> BACKUP 5V; footprint Box IDC header 2x3:Box IDC header 2x3 -> Connector_AMASS:AMASS_XT30U-F_1x02_P5.0mm_Vertical
- U1: value DC-DC_Buck_Converter_7-24V_to_5V_4A -> ~; footprint 2.3 PCBs:DC-DC_Buck_Converter_7-24V_to_5V_4A -> Converter_DCDC:DC-DC Multi-output Buck Converter
- U4: value Adafruit_BNO055_STEMMA_QT -> DEV-16771; footprint 2.3 PCBs:Adafruit IMU BNO055 -> DEV-16771:MODULE_DEV-16771
- moved J13 356.4 mm to (471.4, 180.4), turned to 0 degrees
- moved J12 335.7 mm to (510.3, 118.0), turned to 0 degrees
- moved J6 332.2 mm to (494.9, 119.0), turned to 0 degrees
- moved J22 332.2 mm to (505.7, 118.0), turned to 0 degrees
- moved J3 302.9 mm to (493.6, 149.0), turned to 0 degrees
- moved C1 292.5 mm to (502.9, 141.3), turned to 0 degrees
- moved J19 286.9 mm to (441.0, 170.1)
- moved J20 281.0 mm to (441.0, 177.9)
- moved J15 277.3 mm to (441.0, 138.9)
- moved J18 265.1 mm to (441.0, 162.3), turned to 0 degrees
- moved J7 260.4 mm to (494.9, 126.8)
- moved J14 249.5 mm to (466.8, 180.4)
- moved J16 217.8 mm to (441.0, 146.7)
- moved J17 213.7 mm to (441.0, 154.5)
- moved J11 140.9 mm to (78.8, 175.5), turned to 0 degrees
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Connections:
- C1 pad 1: +5V -> GND
- C1 pad 2: GND -> +3V3
- J1 pad 1: /M1ENCB -> Net-(J1-Pin_1)
- J1 pad 2: /M1ENCA -> GND
- J10 pad 1: Net-(A1-PadNC) -> GND
- J10 pad 2: Net-(A1-PadIOREF) -> +3V3
- J11 pad 1: /DIR1 (1) -> /19
- J11 pad 2: /PWM1 (1) -> /18
- J12 pad 1: +5V -> /13
- J12 pad 2: GND -> /12
- J12 pad 3: /TX -> /11
- J12 pad 4: /RX -> /10
- J12 pad 5: unconnected-(J12-Pad5) -> GND
- J13 pad 1: +5V -> /0
- J13 pad 2: GND -> /1
- J13 pad 3: /SCL -> GND
- J14 pad 1: Net-(A1-PadAD0) -> /19
- J14 pad 2: Net-(A1-PadAD1) -> /18
- J14 pad 3: Net-(A1-PadAD2) -> GND
- J14 pad 4: Net-(A1-PadAD3) -> (no net)
- J15 pad 1: +15V -> +3V3
- J15 pad 2: GND -> /SW1
- J16 pad 1: +15V -> +3V3
- J16 pad 2: GND -> /SW2
- J17 pad 1: Net-(A1-PadAD8) -> +3V3
- J17 pad 2: Net-(A1-PadAD9) -> /SW3
- J18 pad 1: +5V -> +3V3
- J18 pad 2: Net-(A1-Pad23) -> /SW4
- J19 pad 1: Net-(A1-PadSCL) -> +3V3
- J19 pad 2: Net-(A1-PadSDA) -> /SW5
- J2 pad 1: /M2ENCB -> +15V
- J2 pad 2: /M2ENCA -> Net-(J1-Pin_1)
- J20 pad 1: /PWM1 (1) -> +3V3
- J20 pad 2: /PWM2 (2) -> /SW6
- J21 pad 1: /SCL -> GND
- J21 pad 2: /SDA -> /0
- J21 pad 3: /M1ENCA -> /1
- J21 pad 4: /M2ENCA -> /2
- J21 pad 5: /RX -> /3
- J21 pad 6: /TX -> /4
- J21 pad 7: Net-(A1-Pad15) -> /5
- J21 pad 8: Net-(A1-Pad14) -> /6
- J22 pad 1: +5V -> /ON/OFF
- J22 pad 2: /M1ENCB -> /PROGRAM
- J22 pad 3: /M2ENCB -> GND
- J22 pad 4: /M3ENCB -> unconnected-(J22-Pin_4-Pad4)
- J22 pad 5: /M4ENCB -> unconnected-(J22-Pin_5-Pad5)
- J23 pad 1: Net-(A1-PadAD6) -> +5V
- J23 pad 2: Net-(A1-PadAD7) -> GND
- J23 pad 3: Net-(A1-PadAD8) -> +3V3
- J23 pad 4: Net-(A1-PadAD9) -> /23
- J23 pad 5: Net-(A1-PadAD10) -> /22
- J23 pad 6: Net-(A1-PadAD11) -> /21
- J3 pad 1: /M3ENCB -> +15V
- J3 pad 2: /M3ENCA -> GND
- J4 pad 1: /M4ENCB -> Net-(J4-Pin_1)
- J4 pad 2: /M4ENCA -> Net-(J4-Pin_2)
- J4 pad 3: +5V -> Net-(J4-Pin_3)
- J4 pad 4: GND -> unconnected-(J4-Pin_4-Pad4)
- J6 pad 1: +15V -> Net-(J4-Pin_3)
- J6 pad 2: GND -> Net-(J4-Pin_2)
- J9 pad 1: Net-(A1-PadAD0) -> GND
- J9 pad 2: Net-(A1-PadAD1) -> +5V
- U1 pad 4: +5V -> +3V3
- U4 pad 1: +5V -> /1
- U4 pad 10: unconnected-(U4-Pad10) -> /10
- U4 pad 2: unconnected-(U4-Pad2) -> /2
- U4 pad 3: GND -> /3
- U4 pad 4: /SCL -> /4
- U4 pad 5: /SDA -> /5
- U4 pad 6: /RST -> /6
- U4 pad 7: unconnected-(U4-Pad7) -> /7
- U4 pad 8: unconnected-(U4-Pad8) -> /8
- U4 pad 9: unconnected-(U4-Pad9) -> /9
Routing:
- net Net-(J7-PadN): track 239.2 -> 0.00 mm
- net /SDA: track 192.6 -> 0.00 mm, vias 1 -> 0
- net /SCL: track 179.9 -> 0.00 mm, vias 2 -> 0
- net /TX: track 168.8 -> 0.00 mm, vias 1 -> 0
- net /RX: track 165.6 -> 0.00 mm
- net Net-(A1-PadAD6): track 161.1 -> 0.00 mm
- net Net-(A1-PadAD7): track 156.3 -> 0.00 mm
- net Net-(A1-PadAD3): track 152.7 -> 0.00 mm
- net Net-(A1-PadAD0): track 152.4 -> 0.00 mm
- net Net-(A1-PadAD8): track 151.5 -> 0.00 mm, vias 2 -> 0
- net Net-(A1-PadAD1): track 149.4 -> 0.00 mm
- net Net-(A1-PadAD5): track 148.5 -> 0.00 mm
- net Net-(A1-PadAD2): track 146.4 -> 0.00 mm
- net Net-(A1-PadAD10): track 145.4 -> 0.00 mm, vias 1 -> 0
- net Net-(A1-PadAD11): track 143.3 -> 0.00 mm
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- removed copper zone on B.Cu, net +5V
- removed copper zone on F.Cu, net GND
Other:
- board size 215 x 206.6 mm -> 200 x 175 mm
- board text removed: "15V"
- board text removed: "3V3"
- board text removed: "5V"
- board text removed: "G V 2"
- board text removed: "GND"
- board text removed: "LINE PCB"
- board text removed: "LOGIC"
- board text removed: "RX"
- board text removed: "SCL"
- board text removed: "SDA"
- board text removed: "SEN1"
- board text removed: "TX"
- board text removed: "X"
