File: Goku _ Vegeta/3.1/Main 3.1 - GV3/Main 3.1.kicad_sch (KiCad schematic)
At the start: 100 parts, among them J1 BATTERY POWER, J10 Motor 4, J11 LEFT HEADERS, J12 RIGHT HEADERS, J13 MID HEADERS, J2 BACKUP 5V, J3 BACKUP 3V3, J4 I2C, J6 Solenoid, J7 Motor 1, J8 Motor 2, J9 Motor 3, Q1 BSC040N10NS5, U3 LM2587S-ADJ, U4 TB67H420FTG Dual/Single Motor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, U5 TB67H420FTG Dual/Single Motor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, U6 TB67H420FTG Dual/Single Motor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, U7 TB67H420FTG Dual/Single Motor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, U8 DEV-16771

Commit message: MAIN 3.1 DONE no silkscreen
Parts:
- removed A1, A10, A11, A12, A13, A14, A15, A16, A2, A3, A4, A5, A6, A7, A8, A9: ALS-PT19-315C/L177/TR8, ALS-PT19-315C_L177_TR8:XDCR_ALS-PT19-315C_L177_TR8, symbol ALS-PT19-315C_L177_TR8:ALS-PT19-315C/L177/TR8
- removed C1, C11, C14, C9: 100uF, Capacitor_THT:CP_Radial_D10.0mm_P5.00mm, symbol Device:C_Polarized_Small
- removed C10: 1uF, Capacitor_SMD:C_0805_2012Metric, symbol Device:C_Polarized_Small
- removed C12, C13: 560uF, Capacitor_THT:CP_Radial_D18.0mm_P7.50mm, symbol Device:C_Polarized
- removed D3: SS510, Diode_SMD:D_SMC, symbol Device:D_Schottky
- removed J1: BATTERY POWER, Connector_AMASS:AMASS_XT30U-F_1x02_P5.0mm_Vertical, symbol Connector:Conn_01x02_Male
- removed L3: 56uH, Inductor_SMD:L_Bourns_SRR1260, symbol Device:L
- removed LED1, LED10, LED11, LED12, LED13, LED14, LED15, LED16, LED2, LED3, LED4, LED5, LED6, LED7, LED8, LED9: JB2835AWT-W-U30GA0000-N0000001, JB2835AWT-W-U30GA0000-N0000001:LED_J2835_CRW, symbol JB2835AWT-W-U30GA0000-N0000001:JB2835AWT-W-U30GA0000-N0000001
- removed R1, R17, R18, R19, R2, R20, R21, R22, R23, R24, R3, R4, R5, R6, R7, R8: 12R, Resistor_SMD:R_0805_2012Metric, symbol Device:R_Small_US
- removed R10, R11, R12, R13, R14, R15, R16, R25, R26, R27, R28, R29, R30, R31, R32, R9: 10K, Resistor_SMD:R_0805_2012Metric, symbol Device:R_Small_US
- removed R35: 2K94, Resistor_SMD:R_0805_2012Metric, symbol Device:R_Small
- removed R36: 1K5, Resistor_SMD:R_0805_2012Metric, symbol Device:R_Small
- removed R37: CT6EP103, POT_CT-6EP_NDC:POT_CT-6EP_NDC, symbol POT_CT-6EP_NDC:CT6EP103
- removed R38: 57K, Resistor_SMD:R_0805_2012Metric, symbol Device:R_Small
- removed U1: ~, Converter_DCDC:DC-DC Multi-output Buck Converter, symbol Converter_DCDC:DC-DC_Multi-output_Buck_Converter
- removed U3: LM2587S-ADJ, LM2587S-ADJ:VREG_TPS79625KTTR, symbol LM2587S-ADJ:LM2587S-ADJ
- added C1, C7: 10uF, Capacitor_SMD:C_0805_2012Metric, symbol Device:C_Small
- added C3, C4, C5, C6: 750uF, Capacitor_THT:CP_Radial_D10.0mm_P5.00mm, symbol Device:C_Polarized
- added D1: LED, LED_THT:LED_D3.0mm, symbol Device:LED
- added J1: Battery Buzzer, Connector_PinHeader_2.54mm:PinHeader_1x09_P2.54mm_Vertical, symbol Connector:Conn_01x09_Pin
- added J14: UART, Connector_PinSocket_2.54mm:PinSocket_1x03_P2.54mm_Vertical, symbol Connector:Conn_01x03_Socket
- added J15: I2C, Connector_PinSocket_2.54mm:PinSocket_1x03_P2.54mm_Vertical, symbol Connector:Conn_01x03_Socket
- added J16: 4S Battery, Connectors:DEANS, symbol Connector:Conn_01x02_Pin
- added J17: Power Switch, Connector_AMASS:AMASS_XT30UPB-F_1x02_P5.0mm_Vertical, symbol Connector:Conn_01x02_Pin
- added J18: Batt Bal, Connector_JST:JST_XH_B5B-XH-A_1x05_P2.50mm_Vertical, symbol Connector:Conn_01x05_Socket
- added J19: 5V PI, Connector_Wire:SolderWire-0.75sqmm_1x02_P4.8mm_D1.25mm_OD2.3mm, symbol Connector:Conn_01x02_Socket
- added J20: ESC PWR, Connector_AMASS:AMASS_XT30UPB-F_1x02_P5.0mm_Vertical, symbol Connector:Conn_01x02_Pin
- added J23: ESC PWM, Connector_PinHeader_2.54mm:PinHeader_1x03_P2.54mm_Vertical, symbol Connector_Generic:Conn_01x03
- added J5: SPI, Connector_PinSocket_2.54mm:PinSocket_1x05_P2.54mm_Vertical, symbol Connector:Conn_01x05_Socket
- added Q2: Q_Photo_NPN, LED_THT:LED_D3.0mm, symbol Device:Q_Photo_NPN
- added R1, R3, R5, R7: 30R, Resistor_SMD:R_0805_2012Metric, symbol Device:R_Small
- added R10, R11, R12, R14, R2, R4, R6, R9: 10K, Resistor_SMD:R_0805_2012Metric, symbol Device:R_Small
- added R13: 95R, Resistor_SMD:R_0805_2012Metric, symbol Device:R_Small
- added R15: 4R7, Resistor_THT:R_Axial_Power_L25.0mm_W9.0mm_P30.48mm, symbol Device:R
- added U1: ~, Converter_DCDC:Pololu 3.3V, 500mA Step-Down Voltage Regulator D24V5F3, symbol Converter_DCDC:Pololu_3.3V,_500mA_Step-Down_Voltage_Regulator_D24V5F3_
- added U10, U11, U12, U3: ~, Button_Switch_Keyboard:SW_Cherry_MX_3mmLED, symbol Switch:CherryMX_LED
- added U13: Adafruit_BNO055_STEMMA_QT, 2.3 PCBs:Adafruit IMU BNO055, symbol Adafruit BNO055 STEMMA QT:Adafruit_BNO055_STEMMA_QT
- added U14: ~, Converter_DCDC:5V, 5.5A Step-Down Voltage Regulator D36V50F5, symbol Converter_DCDC:5V,_5.5A_Step-Down_Voltage_Regulator_D36V50F5_
- added U9: Arduino Compatible DC-DC Boost Module with Display, Converter_DCDC:Arduino Compatible DC-DC Boost Module with Display, symbol Converter_DCDC:Arduino_Compatible_DC-DC_Boost_Module_with_Display_
- J2: value BACKUP 5V -> 5V LINE
- J3: footprint Connector_AMASS:AMASS_XT30U-F_1x02_P5.0mm_Vertical -> Connector_Wire:SolderWire-0.75sqmm_1x02_P4.8mm_D1.25mm_OD2.3mm
- J6: footprint TerminalBlock:TerminalBlock_bornier-2_P5.08mm -> Connector_Wire:SolderWire-0.75sqmm_1x02_P4.8mm_D1.25mm_OD2.3mm
Connections:
- net +15V: now also J17.1 (Pin_1), J20.2 (Pin_2), U1.2 (VIN), U14.3 (VIN), U9.1 (VIN+)
- net +3V3: now also C1.1, C7.1, Q2.1 (C), R10.2, R11.2, R12.2, R9.2, U1.4 (VOUT), U10.S1, U11.S1, U13.1 (VIN), U3.S1; no longer J11.15 (Pin_15), J12.3 (Pin_3)
- net +5V: now also C2.1, J23.1 (Pin_1), R13.1, U10.A, U11.A, U12.A, U3.A; no longer C2.2
- net 0: now also J14.1 (Pin_1)
- net 1: now also J14.2 (Pin_2)
- net 10: now also J5.4 (Pin_4); no longer U5.5 (INA2)
- net 11: now also J5.3 (Pin_3); no longer U5.4 (INA1)
- net 12: now also J5.2 (Pin_2)
- net 13: now also J5.1 (Pin_1); no longer Q1.4 (G)
- net 16: now also R11.1, U13.4 (SCL)
- net 17: now also R12.1, U13.5 (SDA)
- net 18: now also J15.2 (Pin_2), R10.1
- net 19: now also J15.1 (Pin_1), R9.1
- net 23: now also R2.1, U3.S2 (S1)
- net 24: now also R4.1, U10.S2 (S1)
- net 25: now also R6.1, U11.S2 (S1)
- net 39: now also U5.5 (INA2)
- net 40: now also Q1.4 (G)
- net 41: now also U5.4 (INA1)
- net GND: now also C2.2, C1.2, C3.2, C4.2, C5.2, C6.2, C7.2, D1.1 (K), J14.3 (Pin_3), J15.3 (Pin_3), J16.2 (Pin_2), J19.1 (Pin_1), J20.1 (Pin_1), J23.3 (Pin_3), J5.5 (Pin_5), R1.1, R14.2, R2.2, R3.1, R4.2, R5.1, R6.2, R7.1, U1.3 (GND), U12.S1, U13.3 (GND), U14.2 (GND), U9.2 (VIN-), U9.4 (OUT-); no longer C2.1
- net PROGRAM: now also U12.S2 (S1)
- net at D4.3 (A), J6.1 (Pin_1): now also C3.1, C4.1, C5.1, C6.1, R15.1
- net 3.3V_1: now reaches U8.3.3V_1 (3.3V)
- net 3.3V_1: now also J11.15 (Pin_15)
- net 3.3V_2: now reaches U8.3.3V_2 (3.3V__1)
- net 3.3V_2: now also J12.3 (Pin_3)
- new net: J1.1 (Pin_1), J18.1 (Pin_1)
- new net: J1.2 (Pin_2), J18.2 (Pin_2)
- new net: J1.3 (Pin_3), J18.3 (Pin_3)
- new net: J1.4 (Pin_4), J18.4 (Pin_4)
- new net: J1.5 (Pin_5), J18.5 (Pin_5)
- new net: D1.2 (A), R13.2
- new net: R7.2, U12.K
- new net: R15.2, U9.3 (OUT+)
- new net: R3.2, U10.K
- new net: J19.2 (Pin_2), U14.1 (Vout)
- new net: R5.2, U11.K
- new net: J16.1 (Pin_1), J17.2 (Pin_2)
- new net: R1.2, U3.K
- new net LINE BREAK: Q2.2 (E), R14.1
- new net RST: U13.6 (RST)
- no-connect marks 54 -> 66
Other:
- note added: "3V3 Power Rail - Sensors"
- note added: "5V Power Rail - MCU & Peripherals"
- note added: "5V Power Rail - Rasp Pi and Oak 1"
- note added: "BATTERY"
- note added: "CAM BUS(s)"
- note added: "Kicker Test"
- note added: "LINE BREAK CIRCUIT"
- note added: "LOGIC SWITCHES"
- note added: "NEXT STEPS: MAYBE:"
- note added: "Program"
- note added: "Reset"
- note added: "SENSORS"
- note added: "Start"
- note removed: "2nd Warning Line Sensors - Conditional Poll"
- note removed: "3V3 POWER RAIL - LEDs and Phototransistors"
- note removed: "5V POWER RAIL - Microcontroller"
- note removed: "Boost Circuit"
- note removed: "LINE SENSORS"
- note removed: "NEXT STEPS: add footprint for motor drivers finish adding in footprints for inductors etc. MAYBE:"
- note removed: "Warning Line Sensors - Constant Poll"
- moved on the sheet: D4, J10, J11, J12, J13, J2, J3, J4, J6, J7, J8, J9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

Commit message: Main and Line 3.1 done w/ silkscreen
Parts:
- removed J2: 5V LINE, Connector_AMASS:AMASS_XT30U-F_1x02_P5.0mm_Vertical, symbol Connector:Conn_01x02_Male
- removed J4: I2C, Connector_AMASS:AMASS_XT30U-F_1x02_P5.0mm_Vertical, symbol Connector:Conn_01x02_Male
- added C8, C9: 10uF, Capacitor_SMD:C_0805_2012Metric, symbol Device:C_Small
- added J21: Line, Connector_JST:JST_XH_B4B-XH-A_1x04_P2.50mm_Vertical, symbol Connector_Generic:Conn_01x04
- added R16, R8: 15R, Resistor_THT:R_Axial_DIN0207_L6.3mm_D2.5mm_P10.16mm_Horizontal, symbol Device:R
- added U15: Bluetooth_Module_(HC-05), Connector_PinHeader_2.54mm:PinHeader_1x06_P2.54mm_Vertical, symbol RF_Bluetooth:Bluetooth_Module_(HC-05)
- added U16: Bluetooth_Module_(HC-06), Connector_PinHeader_2.54mm:PinHeader_1x04_P2.54mm_Vertical, symbol RF_Bluetooth:Bluetooth_Module_(HC-06)
- J20: footprint Connector_AMASS:AMASS_XT30UPB-F_1x02_P5.0mm_Vertical -> Connector_Wire:SolderWire-0.5sqmm_1x02_P4.6mm_D0.9mm_OD2.1mm
- R15: value 4R7 -> 15R; footprint Resistor_THT:R_Axial_Power_L25.0mm_W9.0mm_P30.48mm -> Resistor_THT:R_Axial_DIN0207_L6.3mm_D2.5mm_P10.16mm_Horizontal
Connections:
- net +5V: now also C8.1, C9.1, J21.1 (Pin_1), U15.2 (VCC), U16.1 (VCC)
- net 14: now also U15.5 (RX)
- net 15: now also U15.4 (TX)
- net 18: now also J21.3 (Pin_3)
- net 19: now also J21.4 (Pin_4)
- net 20: now also U16.4 (RX)
- net 21: now also U16.3 (TX)
- net 27: now also U15.6 (State)
- net 38: now also U15.1 (EN)
- net GND: now also C8.2, C9.2, J21.2 (Pin_2), U15.3 (GND), U16.2 (GND)
- net at R15.2, U9.3 (OUT+): now also R16.2, R8.2
- net at C3.1, C4.1, C5.1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: now also R16.1, R8.1
Other:
- note added: "BLUETOOTH"
- note added: "MASTER"
- note added: "NEXT STEPS: -need to add bluetooth chip -route wires to pwm on teensy 4.1 MAYBE:"
- note added: "SLAVE"
- note removed: "NEXT STEPS: MAYBE:"
- moved on the sheet: C1, C2, C3, C4, C5, C6, C7, D1, D4, J1, J10, J11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

Commit message: main 3.1 edit actualy done now i think...
Connections:
- net +3V3: now also U10.A, U11.A, U12.A, U3.A
- net +5V: no longer J23.1 (Pin_1), U10.A, U11.A, U12.A, U3.A
- net 22: now also J23.1 (Pin_1)
Changed lines of the file:
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@@
   (junction (at 410.21 63.5) (diameter 0) (color 0 0 0 0)
   )
+  (junction (at 207.01 46.99) (diameter 0) (color 0 0 0 0)
+  )
   (junction (at 83.82 96.52) (diameter 0) (color 0 0 0 0)
   )
@@
   (junction (at 309.88 57.15) (diameter 0) (color 0 0 0 0)
   )
+  (junction (at 207.01 63.5) (diameter 0) (color 0 0 0 0)
+  )
   (junction (at 327.66 57.15) (diameter 0) (color 0 0 0 0)
   )
@@
   (junction (at 279.4 90.17) (diameter 0) (color 0 0 0 0)
   )
+  (junction (at 207.01 30.48) (diameter 0) (color 0 0 0 0)
+  )
   (junction (at 410.21 154.94) (diameter 0) (color 0 0 0 0)
   )
@@
     (stroke (width 0) (type default))
   )
+  (wire (pts (xy 207.01 63.5) (xy 207.01 80.01))
+    (stroke (width 0) (type default))
+  )
   (wire (pts (xy 229.87 30.48) (xy 233.68 30.48))
     (stroke (width 0) (type default))
@@
     (stroke (width 0) (type default))
   )
-  (wire (pts (xy 124.46 63.5) (xy 124.46 60.96))
-    (stroke (width 0) (type default))
-  )
-  (wire (pts (xy 119.38 63.5) (xy 124.46 63.5))
-    (stroke (width 0) (type default))
-  )
   (wire (pts (xy 524.51 135.89) (xy 539.75 135.89))
     (stroke (width 0) (type default))
@@
     (stroke (width 0) (type default))
   )
+  (wire (pts (xy 207.01 24.13) (xy 207.01 30.48))
+    (stroke (width 0) (type default))
+  )
   (wire (pts (xy 524.51 52.07) (xy 533.4 52.07))
     (stroke (width 0) (type default))
@@
     (stroke (width 0) (type default))
   )
+  (wire (pts (xy 207.01 46.99) (xy 207.01 63.5))
+    (stroke (width 0) (type default))
+  )
   (wire (pts (xy 224.79 46.99) (xy 223.52 46.99))
     (stroke (width 0) (type default))
@@
     (stroke (width 0) (type default))
   )
+  (wire (pts (xy 207.01 30.48) (xy 207.01 46.99))
+    (stroke (width 0) (type default))
+  )
   (wire (pts (xy 85.09 66.04) (xy 96.52 66.04))
     (stroke (width 0) (type default))
@@
     (stroke (width 0) (type default))
   )
+  (wire (pts (xy 119.38 63.5) (xy 128.27 63.5))
+    (stroke (width 0) (type default))
+  )
   (wire (pts (xy 415.29 152.4) (xy 415.29 154.94))
     (stroke (width 0) (type default))
@@
     (effects (font (size 1.27 1.27)) (justify left bottom))
   )
+  (label "ESCPWM" (at 128.27 63.5 180) (fields_autoplaced)
+    (effects (font (size 1.27 1.27)) (justify right bottom))
+  )
   (label "40" (at 527.05 123.19 180) (fields_autoplaced)
     (effects (font (size 1.27 1.27)) (justify right bottom))
@@
     (effects (font (size 1.27 1.27)) (justify right bottom))
   )
+  (label "ESCPWM" (at 471.17 135.89 0) (fields_autoplaced)
+    (effects (font (size 1.27 1.27)) (justify left bottom))
+  )
   (label "TX3" (at 261.62 50.8 90) (fields_autoplaced)
     (effects (font (size 1.27 1.27)) (justify left bottom))
@@
     )
   )
-  (symbol (lib_name "+5V_3") (lib_id "power:+5V") (at 207.01 46.99 0) (unit 1)
-    (in_bom yes) (on_board yes) (dnp no)
-    (property "Reference" "#PWR032" (at 207.01 50.8 0)
-      (effects (font (size 1.27 1.27)) hide)
-    )
-    (property "Value" "+5V" (at 207.01 43.18 0)
-      (effects (font (size 1.27 1.27)))
-    )
-    (property "Footprint" "" (at 207.01 46.99 0)
-      (effects (font (size 1.27 1.27)) hide)
-    )
-    (property "Datasheet" "" (at 207.01 46.99 0)
-      (effects (font (size 1.27 1.27)) hide)
-    )
-    (pin "1")
-    (instances
-      (project "Main 3.1"
-        (path "/d5c7bd24-918a-4dd6-9ba7-d38579daba08"
-          (reference "#PWR032") (unit 1)
-        )
-      )
-    )
-  )
   (symbol (lib_id "power:GND") (at 161.29 36.83 0) (unit 1)
     (in_bom yes) (on_board yes) (dnp no)
@@
     )
   )
+  (symbol (lib_id "power:+3V3") (at 207.01 24.13 0) (unit 1)
+    (in_bom yes) (on_board yes) (dnp no)
+    (property "Reference" "#PWR025" (at 207.01 27.94 0)
+      (effects (font (size 1.27 1.27)) hide)
+    )
+    (property "Value" "+3V3" (at 207.01 20.32 0)
+      (effects (font (size 1.27 1.27)))
+    )
+    (property "Footprint" "" (at 207.01 24.13 0)
+      (effects (font (size 1.27 1.27)) hide)
+    )
+    (property "Datasheet" "" (at 207.01 24.13 0)
+      (effects (font (size 1.27 1.27)) hide)
+    )
+    (pin "1")
+    (instances
+      (project "Main 3.1"
+        (path "/d5c7bd24-918a-4dd6-9ba7-d38579daba08"
+          (reference "#PWR025") (unit 1)
+        )
+      )
+    )
+  )
   (symbol (lib_id "Device:C_Polarized_Small") (at 97.79 34.29 0) (mirror y) (unit 1)
     (in_bom yes) (on_board yes) (dnp no)
@@
     )
   )
-  (symbol (lib_name "+5V_3") (lib_id "power:+5V") (at 207.01 30.48 0) (unit 1)
-    (in_bom yes) (on_board yes) (dnp no)
-    (property "Reference" "#PWR033" (at 207.01 34.29 0)
-      (effects (font (size 1.27 1.27)) hide)
-    )
-    (property "Value" "+5V" (at 207.01 26.67 0)
-      (effects (font (size 1.27 1.27)))
-    )
-    (property "Footprint" "" (at 207.01 30.48 0)
-      (effects (font (size 1.27 1.27)) hide)
-    )
-    (property "Datasheet" "" (at 207.01 30.48 0)
-      (effects (font (size 1.27 1.27)) hide)
-    )
-    (pin "1")
-    (instances
-      (project "Main 3.1"
-        (path "/d5c7bd24-918a-4dd6-9ba7-d38579daba08"
-          (reference "#PWR033") (unit 1)
-        )
-      )
-    )
-  )
   (symbol (lib_id "power:GND") (at 233.68 66.04 0) (unit 1)
     (in_bom yes) (on_board yes) (dnp no)
@@
     )
   )
-  (symbol (lib_name "+5V_3") (lib_id "power:+5V") (at 207.01 80.01 0) (unit 1)
-    (in_bom yes) (on_board yes) (dnp no)
-    (property "Reference" "#PWR030" (at 207.01 83.82 0)
-      (effects (font (size 1.27 1.27)) hide)
-    )
-    (property "Value" "+5V" (at 207.01 76.2 0)
-      (effects (font (size 1.27 1.27)))
-    )
-    (property "Footprint" "" (at 207.01 80.01 0)
-      (effects (font (size 1.27 1.27)) hide)
-    )
-    (property "Datasheet" "" (at 207.01 80.01 0)
-      (effects (font (size 1.27 1.27)) hide)
-    )
-    (pin "1")
-    (instances
-      (project "Main 3.1"
-        (path "/d5c7bd24-918a-4dd6-9ba7-d38579daba08"
-          (reference "#PWR030") (unit 1)
-        )
-      )
-    )
-  )
   (symbol (lib_id "power:+15V") (at 66.04 24.13 0) (unit 1)
     (in_bom yes) (on_board yes) (dnp no)
@@
     )
   )
-  (symbol (lib_name "+5V_2") (lib_id "power:+5V") (at 124.46 60.96 0) (unit 1)
-    (in_bom yes) (on_board yes) (dnp no)
-    (property "Reference" "#PWR025" (at 124.46 64.77 0)
-      (effects (font (size 1.27 1.27)) hide)
-    )
-    (property "Value" "+5V" (at 124.46 57.15 0)
-      (effects (font (size 1.27 1.27)))
-    )
-    (property "Footprint" "" (at 124.46 60.96 0)
-      (effects (font (size 1.27 1.27)) hide)
-    )
-    (property "Datasheet" "" (at 124.46 60.96 0)
-      (effects (font (size 1.27 1.27)) hide)
-    )
-    (pin "1")
-    (instances
-      (project "Main 3.1"
-        (path "/d5c7bd24-918a-4dd6-9ba7-d38579daba08"
-          (reference "#PWR025") (unit 1)
-        )
-      )
-    )
-  )
   (symbol (lib_id "Device:R_Small") (at 227.33 30.48 270) (unit 1)
     (in_bom yes) (on_board yes) (dnp no)
@@
         )
       )
-    )
-  )
-  (symbol (lib_name "+5V_3") (lib_id "power:+5V") (at 207.01 63.5 0) (unit 1)
-    (in_bom yes) (on_board yes) (dnp no)
-    (property "Reference" "#PWR031" (at 207.01 67.31 0)
-      (effects (font (size 1.27 1.27)) hide)
-    )
-    (property "Value" "+5V" (at 207.01 59.69 0)
-      (effects (font (size 1.27 1.27)))
-    )
-    (property "Footprint" "" (at 207.01 63.5 0)
-      (effects (font (size 1.27 1.27)) hide)
-    )
-    (property "Datasheet" "" (at 207.01 63.5 0)
-      (effects (font (size 1.27 1.27)) hide)
-    )
-    (pin "1")
-    (instances
-      (project "Main 3.1"
-        (path "/d5c7bd24-918a-4dd6-9ba7-d38579daba08"
-          (reference "#PWR031") (unit 1)
-        )
-      )

Commit message: kjwefqkwenfqerlgk
Connections:
- net LINE BREAK is gone; now on net 26: Q2.2 (E), R14.1
Changed lines of the file:
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@@
     (effects (font (size 1.27 1.27)) (justify left bottom))
+  )
+  (label "LINE BREAK" (at 539.75 133.35 180) (fields_autoplaced)
+    (effects (font (size 1.27 1.27)) (justify right bottom))
   )
   (label "35" (at 544.83 121.92 0) (fields_autoplaced)
