File: SumoBot/2.1/SumoNyx2.1/SumoNyx2.1.kicad_sch (KiCad schematic)
At the start: 17 parts, among them J1 SW, J2 BATT, J3 Motor 1, J4 BACK LED, J5 Motor 2, J6 Eyes I2C, Q1 AO3422, U2 AZ1117-5.0, U3 DRV8833BRKT, U4 NRF24L01_SMD_Module

Commit message: commit b4 sleep
Parts:
- removed U3: DRV8833BRKT, DRV8833BRKT:DRV8833BRKT, symbol DRV8833BRKT:DRV8833BRKT
- removed U4: NRF24L01_SMD_Module, symbol RF_Module:NRF24L01_SMD_Module
- added U1: NRF24L01_SMD_Module, RF_Module:NRF24L01_SMD_Module, symbol RF_Module:NRF24L01_SMD_Module
- added U3: DRV8833_Module, symbol Driver_Motor:DRV8833_Module
Connections:
- net AIN1: now also U3.12 (AIN1)
- net AIN2: now also U3.11 (AIN2)
- net BIN1: now also U3.7 (BIN1)
- net BIN2: now also U3.6 (nFAULT)
- net CE: now also U1.3 (CE)
- net CSN: now also U1.4 (CSN)
- net GND: now also U1.2 (Vss(GND)), U3.8 (GND)
- net MISO: now also U1.7 (MISO)
- net MOSI: now also U1.6 (MOSI)
- net SCK: now also U1.5 (SCK)
- net at J3.1 (Pin_1): now also U3.4 (BOUT1)
- net at J3.2 (Pin_2): now also U3.5 (BOUT2)
- net at J5.1 (Pin_1): now also U3.2 (AOUT2)
- net at J5.2 (Pin_2): now also U3.3 (AOUT1)
- net +3.3V renamed +3V3
- net +3V3: now also U1.1 (Vdd(3V3))
- net +7.5V renamed +8V
- net +8V: now also U3.9 (VM)
Other:
- moved on the sheet: A1, J3, J5

Commit message: kjwefqkwenfqerlgk
Parts:
- added J7: 2s Lipo Balance, Connector_JST:JST_XH_B3B-XH-A_1x03_P2.50mm_Vertical, symbol Connector:Conn_01x03_Pin
Connections:
- net GND: now also J7.1 (Pin_1)
Other:
- moved on the sheet: A1, C1, C2, C3, F1, J3, J4, J5, J6, R2, U1, U2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
