File: Goku _ Vegeta/4.4/Line 4.4/Line 4.3.kicad_pcb (KiCad board)
At the start: 2 copper layers, 135 x 126 mm, 143 parts, among them J1 Line, U1 AP63203WU, U3 LM339, U4 LM339, U5 LM339, U6 LM339, U7 LM339, U8 LM339, U9 ESP32-DEVKITC-32U

Commit message: lol
Other:
- outline, holes or cut-outs redrawn
