File: Self_Balancing_Robot/SBRcontroller/SBRcontroller.kicad_pcb (KiCad board)
At the start: 2 copper layers, 113.5 x 60.8 mm, 28 parts, among them J2 -SW, J3 +SW, J4 +SWLED, J5 -SWLED, U1 THB001P, U11 THB001P, U7 ESP32-DEVKITC

Commit message: lol
Connections:
- U7 pad 10: /P2H -> unconnected-(U7-IO26-Pad10)
- U7 pad 11: /P2V -> unconnected-(U7-IO27-Pad11)
- U7 pad 12: /P1H -> unconnected-(U7-IO14-Pad12)
- U7 pad 13: /P1V -> unconnected-(U7-IO12-Pad13)
- U7 pad 14: unconnected-(U7-GND1-Pad14) -> GND
- U7 pad 38: unconnected-(U7-GND3-Pad38) -> GND
- U7 pad 6: unconnected-(U7-IO35-Pad6) -> /P2H
- U7 pad 7: unconnected-(U7-IO32-Pad7) -> /P2V
- U7 pad 8: unconnected-(U7-IO33-Pad8) -> /P1H
- U7 pad 9: unconnected-(U7-IO25-Pad9) -> /P1V
Routing:
- net /P1H: track 20.3 -> 12.4 mm
- net /P2V: track 57.2 -> 50.0 mm
- net /P2H: track 44.8 -> 37.7 mm, vias 1 -> 0
- net /SW1: track 61.3 -> 57.2 mm
- net /KB2: track 61.5 -> 63.7 mm
- net /P1V: track 6.88 -> 5.78 mm
