File: Self_Balancing_Robot/SBR2.1/SBR2.kicad_sch (KiCad schematic)
At the start: 26 parts, among them J1 Conn_01x02, J2 Conn_01x04, J3 Conn_01x04, J4 +SW, J5 -SW, J6 +SWLED, J7 -SWLED, J8 Conn_01x05, J9 Conn_01x05, U1 A4988_STEPPER_MOTOR_DRIVER_CA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, U2 A4988_STEPPER_MOTOR_DRIVER_CA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, U3 ESP32-DEVKITC, U4 NCP1117-5.0_SOT223, U6 Adafruit IMU BNO055

Commit message: what is happening
Other:
- note added: "need to update"
Changed lines of the file:
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@@
+		)
+	)
+	(text "need to update"
+		(exclude_from_sim no)
+		(at 50.038 211.836 0)
+		(effects
+			(font
+				(size 1.27 1.27)
+			)
 		)
 	)
