File: Self_Balancing_Robot/SBR2.1/SBR2.1.kicad_pcb (KiCad board)
At the start: 2 copper layers, 88 x 64 mm, 28 parts, among them J1 Conn_01x02, J2 Conn_01x04, J3 Conn_01x04, J4 +SW, J5 -SW, J6 +SWLED, J7 -SWLED, J8 Conn_01x05, J9 Conn_01x05, U1 A4988_STEPPER_MOTOR_DRIVER_CA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, U2 A4988_STEPPER_MOTOR_DRIVER_CA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, U3 ESP32-DEVKITC, U4 NCP1117-5.0_SOT223, U6 Adafruit IMU BNO055

Commit message: pcb mfr
Parts:
- removed J5: -SW, SparkFun-Connector:1x01
- removed J6: +SWLED, SparkFun-Connector:1x01
- removed J7: -SWLED, SparkFun-Connector:1x01
- removed U4: NCP1117-5.0_SOT223, Package_TO_SOT_SMD:SOT-223-3_TabPin2
- added U5: uA7805, Package_TO_SOT_SMD:TO-263-3_TabPin2, F.Cu at (149.9, 65.3)
- D1: value D_Zener -> 1N5243BTR
- J4: value +SW -> Conn_01x04; footprint SparkFun-Connector:1x01 -> Connector_JST:JST_XH_B4B-XH-AM_1x04_P2.50mm_Vertical; moved to B.Cu
- moved C2 16.9 mm to (139.0, 78.5), turned to -90 degrees
- moved C1 15.0 mm to (139.0, 54.8), turned to 90 degrees
- moved J1 5.06 mm to (159.8, 63.5), turned to -90 degrees
- moved J4 2.25 mm to (130.8, 82.5)
Connections:
- U1 pad 2: unconnected-(U1-MS1-Pad2) -> +5V
- U1 pad 3: unconnected-(U1-MS2-Pad3) -> +5V
- U1 pad 4: unconnected-(U1-MS3-Pad4) -> +5V
- U2 pad 2: unconnected-(U2-MS1-Pad2) -> +5V
- U2 pad 3: unconnected-(U2-MS2-Pad3) -> +5V
- U2 pad 4: unconnected-(U2-MS3-Pad4) -> +5V
Routing:
- net +5V: track 181.6 -> 218.1 mm, vias 0 -> 1
- net GND: track 83.4 -> 47.0 mm, vias 0 -> 20
- net +15V: track 123.1 -> 132.5 mm, vias 13 -> 2
- net Net-(J1-Pin_2): track 39.6 -> 48.5 mm
- removed copper zone on F.Cu, net +15V
Other:
- board text added: "19/9/24"
- board text removed: "15/9/24"
- board text removed: "Make sure to set current limit on drivers before turning on"
