File: Self_Balancing_Robot/SBR2.1/SBR2.1.kicad_sch (KiCad schematic)
At the start: 28 parts, among them J1 Conn_01x02, J2 Conn_01x04, J3 Conn_01x04, J4 +SW, J5 -SW, J6 +SWLED, J7 -SWLED, J8 Conn_01x05, J9 Conn_01x05, U1 A4988_STEPPER_MOTOR_DRIVER_CA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, U2 A4988_STEPPER_MOTOR_DRIVER_CA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, U3 ESP32-DEVKITC, U4 NCP1117-5.0_SOT223, U6 Adafruit IMU BNO055

Commit message: pid
Connections:
- net CS1: now also J9.4 (Pin_4)
- net CS2: no longer names the net of U3.27 (IO16)
- net CS2: no longer J9.4 (Pin_4)
- no-connect marks 38 -> 39
Changed lines of the file:
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@@
+	)
+	(no_connect
+		(at 179.07 54.61)
 	)
 	(no_connect
@@
 		(pts
 			(xy 245.11 90.17) (xy 241.3 90.17)
-		)
-		(stroke
-			(width 0)
-			(type default)
-		)
-	)
-	(wire
-		(pts
-			(xy 187.96 54.61) (xy 179.07 54.61)
 		)
 		(stroke
@@
 		)
 	)
-	(label "CS2"
-		(at 237.49 149.86 0)
-		(fields_autoplaced yes)
-		(effects
-			(font
-				(size 1.27 1.27)
-			)
-			(justify left bottom)
-		)
-	)
 	(label "SDA"
 		(at 111.76 74.93 180)
@@
 		)
 	)
+	(label "CS1"
+		(at 237.49 149.86 0)
+		(fields_autoplaced yes)
+		(effects
+			(font
+				(size 1.27 1.27)
+			)
+			(justify left bottom)
+		)
+	)
 	(label "M1STEP"
 		(at 187.96 57.15 180)
@@
 		)
 	)
-	(label "CS2"
-		(at 187.96 54.61 180)
-		(fields_autoplaced yes)
-		(effects
-			(font
-				(size 1.27 1.27)
-			)
-			(justify right bottom)
-		)
-	)

Commit message: pcb mfr
Parts:
- removed J4: +SW, SparkFun-Connector:1x01, symbol SparkFun-Connector:Conn_01x01
- removed J5: -SW, SparkFun-Connector:1x01, symbol SparkFun-Connector:Conn_01x01
- removed J6: +SWLED, SparkFun-Connector:1x01, symbol SparkFun-Connector:Conn_01x01
- removed J7: -SWLED, SparkFun-Connector:1x01, symbol SparkFun-Connector:Conn_01x01
- removed U4: NCP1117-5.0_SOT223, Package_TO_SOT_SMD:SOT-223-3_TabPin2, symbol Regulator_Linear:NCP1117-5.0_SOT223
- added J4: Conn_01x04, Connector_JST:JST_XH_B4B-XH-AM_1x04_P2.50mm_Vertical, symbol Connector_Generic:Conn_01x04
- added U5: uA7805, Package_TO_SOT_SMD:TO-263-3_TabPin2, symbol Regulator_Linear:uA7805
- D1: value D_Zener -> 1N5243BTR
Connections:
- net +15V: now also J4.1 (Pin_1), U5.1 (IN)
- net +5V: now also U1.2 (MS1), U1.3 (MS2), U1.4 (MS3), U2.2 (MS1), U2.3 (MS2), U2.4 (MS3), J4.2 (Pin_2), U5.3 (OUT)
- net GND: now also J4.4 (Pin_4), U5.2 (GND)
- net at J1.2 (Pin_2): now also J4.3 (Pin_3)
- no-connect marks 39 -> 33
Other:
- note added: "13V Zener + 0.5V = 13.5V to pass through LED turns off @ 13.5V"
- note added: "Switch Connector"
- note removed: "11V Zener + 2.5 Fv on LED = 13.5V to pass through LED turns off @ 13.5V"
- moved on the sheet: J1, J9
