File: Goku _ Vegeta/4.0/linetest4.0/linetest4.0.kicad_sch (KiCad schematic)
At the start: 111 parts, among them J1 Line, U1 AP63203WU, U2 LM339, U3 LM339, U4 LM339, U5 LM339, U6 LM339, U7 SC0915

Commit message: changes
Parts:
- A1, A10, A11, A12, A13, A14, A15, A16, A17, A18, A2, A3, A4, A5, A6, A7, A8, A9: symbol ALS-PT19-315C_L177_TR8:ALS-PT19-315C/L177/TR8 -> ALS-PT19-315C_L177_TR8:ALS-PT19-315C/L177/TR8
